File: BenzKnobz/BenzKnobz.kicad_pcb (KiCad board)
At the start: 2 copper layers, 59 parts, among them U1 Teensy4.0

Commit message: board
pcb
Parts:
- removed the ? at (197.8, 79.5)
- removed the ? at (126.7, 79.5)
- removed the REF** at (101.6, 158.1)
- removed the REF** at (83.9, 140.3)
- removed the REF** at (119.4, 104.8)
- removed the REF** at (190.5, 87.0)
- removed the REF** at (119.4, 87.0)
- removed the REF** at (119.4, 140.3)
- removed the REF** at (190.5, 69.2)
- removed the REF** at (101.6, 122.6)
- removed the REF** at (101.6, 140.3)
- removed the REF** at (101.6, 104.8)
- removed the REF** at (101.6, 69.2)
- removed the REF** at (119.4, 69.2)
- removed the REF** at (83.9, 158.1)
- removed the REF** at (83.9, 69.2)
- removed the REF** at (101.6, 87.0)
- removed the REF** at (190.5, 104.8)
- removed the REF** at (119.4, 122.6)
- removed the REF** at (83.9, 122.6)
- removed the REF** at (83.9, 87.0)
- removed the REF** at (119.4, 158.1)
- removed the REF** at (83.9, 104.8)
- added ?: , , F.Cu at (113.3, 126.9)
- added ?: , , F.Cu at (166.7, 126.9)
- added ?: , , F.Cu at (141.3, 126.9)
- added REF**: LED_SK6812MINI_PLCC4_3.5x3.5mm_P1.75mm, LED_SMD:LED_SK6812MINI_PLCC4_3.5x3.5mm_P1.75mm, F.Cu at (116.8, 113.7)
- added REF**: LED_SK6812MINI_PLCC4_3.5x3.5mm_P1.75mm, LED_SMD:LED_SK6812MINI_PLCC4_3.5x3.5mm_P1.75mm, F.Cu at (144.7, 73.0)
- added REF**: LED_SK6812MINI_PLCC4_3.5x3.5mm_P1.75mm, LED_SMD:LED_SK6812MINI_PLCC4_3.5x3.5mm_P1.75mm, F.Cu at (170.1, 73.0)
- added REF**: LED_SK6812MINI_PLCC4_3.5x3.5mm_P1.75mm, LED_SMD:LED_SK6812MINI_PLCC4_3.5x3.5mm_P1.75mm, F.Cu at (116.8, 134.0)
- added REF**: Potentiometer_Alps_RK09L_Single_Vertical, Potentiometer_THT:Potentiometer_Alps_RK09L_Single_Vertical, F.Cu at (172.7, 17.1)
- added REF**: CONN_MJ-3502, audioJack:CONN_MJ-3502, F.Cu at (132.0, 19.7)
- added REF**: LED_SK6812MINI_PLCC4_3.5x3.5mm_P1.75mm, LED_SMD:LED_SK6812MINI_PLCC4_3.5x3.5mm_P1.75mm, F.Cu at (60.9, 92.7)
- added REF**: LED_SK6812MINI_PLCC4_3.5x3.5mm_P1.75mm, LED_SMD:LED_SK6812MINI_PLCC4_3.5x3.5mm_P1.75mm, F.Cu at (88.8, 133.3)
- added REF**: CONN_MJ-3502, audioJack:CONN_MJ-3502, F.Cu at (104.1, 19.7)
- added REF**: CONN_MJ-3502, audioJack:CONN_MJ-3502, F.Cu at (20.2, 19.0)
- added REF**: Potentiometer_Alps_RK09L_Single_Vertical, Potentiometer_THT:Potentiometer_Alps_RK09L_Single_Vertical, F.Cu at (172.6, 77.5)
- added REF**: LED_SK6812MINI_PLCC4_3.5x3.5mm_P1.75mm, LED_SMD:LED_SK6812MINI_PLCC4_3.5x3.5mm_P1.75mm, F.Cu at (32.9, 92.7)
- added REF**: Potentiometer_Alps_RK09L_Single_Vertical, Potentiometer_THT:Potentiometer_Alps_RK09L_Single_Vertical, F.Cu at (147.2, 118.1)
- added REF**: Potentiometer_Alps_RK09L_Single_Vertical, Potentiometer_THT:Potentiometer_Alps_RK09L_Single_Vertical, F.Cu at (119.3, 77.5)
- added REF**: Potentiometer_Alps_RK09L_Single_Vertical, Potentiometer_THT:Potentiometer_Alps_RK09L_Single_Vertical, F.Cu at (119.3, 36.8)
- added REF**: Potentiometer_Alps_RK09L_Single_Vertical, Potentiometer_THT:Potentiometer_Alps_RK09L_Single_Vertical, F.Cu at (147.2, 36.8)
- added REF**: Potentiometer_Alps_RK09L_Single_Vertical, Potentiometer_THT:Potentiometer_Alps_RK09L_Single_Vertical, F.Cu at (147.2, 57.1)
- added REF**: LED_SK6812MINI_PLCC4_3.5x3.5mm_P1.75mm, LED_SMD:LED_SK6812MINI_PLCC4_3.5x3.5mm_P1.75mm, F.Cu at (32.9, 31.7)
- added REF**: CONN_MJ-3502, audioJack:CONN_MJ-3502, F.Cu at (48.2, 19.0)
- added REF**: LED_SK6812MINI_PLCC4_3.5x3.5mm_P1.75mm, LED_SMD:LED_SK6812MINI_PLCC4_3.5x3.5mm_P1.75mm, F.Cu at (60.9, 133.3)
- added REF**: Potentiometer_Alps_RK09L_Single_Vertical, Potentiometer_THT:Potentiometer_Alps_RK09L_Single_Vertical, F.Cu at (147.2, 97.8)
- added REF**: Potentiometer_Alps_RK09L_Single_Vertical, Potentiometer_THT:Potentiometer_Alps_RK09L_Single_Vertical, F.Cu at (119.3, 57.1)
- added REF**: LED_SK6812MINI_PLCC4_3.5x3.5mm_P1.75mm, LED_SMD:LED_SK6812MINI_PLCC4_3.5x3.5mm_P1.75mm, F.Cu at (144.7, 93.3)
- added REF**: LED_SK6812MINI_PLCC4_3.5x3.5mm_P1.75mm, LED_SMD:LED_SK6812MINI_PLCC4_3.5x3.5mm_P1.75mm, F.Cu at (170.0, 32.4)
- added REF**: LED_SK6812MINI_PLCC4_3.5x3.5mm_P1.75mm, LED_SMD:LED_SK6812MINI_PLCC4_3.5x3.5mm_P1.75mm, F.Cu at (32.9, 52.0)
- added REF**: LED_SK6812MINI_PLCC4_3.5x3.5mm_P1.75mm, LED_SMD:LED_SK6812MINI_PLCC4_3.5x3.5mm_P1.75mm, F.Cu at (60.9, 52.0)
- added REF**: LED_SK6812MINI_PLCC4_3.5x3.5mm_P1.75mm, LED_SMD:LED_SK6812MINI_PLCC4_3.5x3.5mm_P1.75mm, F.Cu at (88.8, 113.0)
- added REF**: LED_SK6812MINI_PLCC4_3.5x3.5mm_P1.75mm, LED_SMD:LED_SK6812MINI_PLCC4_3.5x3.5mm_P1.75mm, F.Cu at (88.8, 52.0)
- added REF**: LED_SK6812MINI_PLCC4_3.5x3.5mm_P1.75mm, LED_SMD:LED_SK6812MINI_PLCC4_3.5x3.5mm_P1.75mm, F.Cu at (60.9, 72.4)
- added REF**: LED_SK6812MINI_PLCC4_3.5x3.5mm_P1.75mm, LED_SMD:LED_SK6812MINI_PLCC4_3.5x3.5mm_P1.75mm, F.Cu at (144.7, 52.7)
- added REF**: LED_SK6812MINI_PLCC4_3.5x3.5mm_P1.75mm, LED_SMD:LED_SK6812MINI_PLCC4_3.5x3.5mm_P1.75mm, F.Cu at (170.1, 154.3)
- added REF**: LED_SK6812MINI_PLCC4_3.5x3.5mm_P1.75mm, LED_SMD:LED_SK6812MINI_PLCC4_3.5x3.5mm_P1.75mm, F.Cu at (60.9, 31.7)
- added REF**: LED_SK6812MINI_PLCC4_3.5x3.5mm_P1.75mm, LED_SMD:LED_SK6812MINI_PLCC4_3.5x3.5mm_P1.75mm, F.Cu at (60.9, 113.0)
- added REF**: LED_SK6812MINI_PLCC4_3.5x3.5mm_P1.75mm, LED_SMD:LED_SK6812MINI_PLCC4_3.5x3.5mm_P1.75mm, F.Cu at (170.1, 134.0)
- added REF**: LED_SK6812MINI_PLCC4_3.5x3.5mm_P1.75mm, LED_SMD:LED_SK6812MINI_PLCC4_3.5x3.5mm_P1.75mm, F.Cu at (32.9, 153.7)
- added REF**: LED_SK6812MINI_PLCC4_3.5x3.5mm_P1.75mm, LED_SMD:LED_SK6812MINI_PLCC4_3.5x3.5mm_P1.75mm, F.Cu at (170.1, 113.7)
- added REF**: Potentiometer_Alps_RK09L_Single_Vertical, Potentiometer_THT:Potentiometer_Alps_RK09L_Single_Vertical, F.Cu at (119.3, 97.8)
- added REF**: Potentiometer_Alps_RK09L_Single_Vertical, Potentiometer_THT:Potentiometer_Alps_RK09L_Single_Vertical, F.Cu at (172.6, 118.1)
- added REF**: Potentiometer_Alps_RK09L_Single_Vertical, Potentiometer_THT:Potentiometer_Alps_RK09L_Single_Vertical, F.Cu at (147.3, 17.1)
- added REF**: LED_SK6812MINI_PLCC4_3.5x3.5mm_P1.75mm, LED_SMD:LED_SK6812MINI_PLCC4_3.5x3.5mm_P1.75mm, F.Cu at (116.8, 154.3)
- added REF**: LED_SK6812MINI_PLCC4_3.5x3.5mm_P1.75mm, LED_SMD:LED_SK6812MINI_PLCC4_3.5x3.5mm_P1.75mm, F.Cu at (144.7, 134.0)
- added REF**: Potentiometer_Alps_RK09L_Single_Vertical, Potentiometer_THT:Potentiometer_Alps_RK09L_Single_Vertical, F.Cu at (147.2, 77.5)
- added REF**: Potentiometer_Alps_RK09L_Single_Vertical, Potentiometer_THT:Potentiometer_Alps_RK09L_Single_Vertical, F.Cu at (172.6, 57.1)
- added REF**: CONN_MJ-3502, audioJack:CONN_MJ-3502, F.Cu at (76.1, 19.0)
- added REF**: LED_SK6812MINI_PLCC4_3.5x3.5mm_P1.75mm, LED_SMD:LED_SK6812MINI_PLCC4_3.5x3.5mm_P1.75mm, F.Cu at (116.8, 52.7)
- added REF**: LED_SK6812MINI_PLCC4_3.5x3.5mm_P1.75mm, LED_SMD:LED_SK6812MINI_PLCC4_3.5x3.5mm_P1.75mm, F.Cu at (32.9, 72.4)
- added REF**: Potentiometer_Alps_RK09L_Single_Vertical, Potentiometer_THT:Potentiometer_Alps_RK09L_Single_Vertical, F.Cu at (119.3, 118.1)
- added REF**: LED_SK6812MINI_PLCC4_3.5x3.5mm_P1.75mm, LED_SMD:LED_SK6812MINI_PLCC4_3.5x3.5mm_P1.75mm, F.Cu at (144.6, 32.4)
- added REF**: LED_SK6812MINI_PLCC4_3.5x3.5mm_P1.75mm, LED_SMD:LED_SK6812MINI_PLCC4_3.5x3.5mm_P1.75mm, F.Cu at (32.9, 113.0)
- added REF**: Potentiometer_Alps_RK09L_Single_Vertical, Potentiometer_THT:Potentiometer_Alps_RK09L_Single_Vertical, F.Cu at (172.6, 36.8)
- added REF**: LED_SK6812MINI_PLCC4_3.5x3.5mm_P1.75mm, LED_SMD:LED_SK6812MINI_PLCC4_3.5x3.5mm_P1.75mm, F.Cu at (88.8, 153.7)
- added REF**: LED_SK6812MINI_PLCC4_3.5x3.5mm_P1.75mm, LED_SMD:LED_SK6812MINI_PLCC4_3.5x3.5mm_P1.75mm, F.Cu at (170.1, 52.7)
- added REF**: KYCON_KCDX-5S-N, midiJack:KYCON_KCDX-5S-N, F.Cu at (-114.3, 152.4)
- added REF**: LED_SK6812MINI_PLCC4_3.5x3.5mm_P1.75mm, LED_SMD:LED_SK6812MINI_PLCC4_3.5x3.5mm_P1.75mm, F.Cu at (88.8, 72.4)
- added REF**: LED_SK6812MINI_PLCC4_3.5x3.5mm_P1.75mm, LED_SMD:LED_SK6812MINI_PLCC4_3.5x3.5mm_P1.75mm, F.Cu at (144.7, 113.7)
- added REF**: LED_SK6812MINI_PLCC4_3.5x3.5mm_P1.75mm, LED_SMD:LED_SK6812MINI_PLCC4_3.5x3.5mm_P1.75mm, F.Cu at (60.9, 153.7)
- added REF**: Potentiometer_Alps_RK09L_Single_Vertical, Potentiometer_THT:Potentiometer_Alps_RK09L_Single_Vertical, F.Cu at (172.6, 97.8)
- added REF**: Potentiometer_Alps_RK09L_Single_Vertical, Potentiometer_THT:Potentiometer_Alps_RK09L_Single_Vertical, F.Cu at (119.3, 138.4)
- added REF**: LED_SK6812MINI_PLCC4_3.5x3.5mm_P1.75mm, LED_SMD:LED_SK6812MINI_PLCC4_3.5x3.5mm_P1.75mm, F.Cu at (32.9, 133.3)
- added REF**: LED_SK6812MINI_PLCC4_3.5x3.5mm_P1.75mm, LED_SMD:LED_SK6812MINI_PLCC4_3.5x3.5mm_P1.75mm, F.Cu at (170.1, 93.3)
- added REF**: LED_SK6812MINI_PLCC4_3.5x3.5mm_P1.75mm, LED_SMD:LED_SK6812MINI_PLCC4_3.5x3.5mm_P1.75mm, F.Cu at (116.7, 32.4)
- added REF**: LED_SK6812MINI_PLCC4_3.5x3.5mm_P1.75mm, LED_SMD:LED_SK6812MINI_PLCC4_3.5x3.5mm_P1.75mm, F.Cu at (144.7, 154.3)
- added REF**: LED_SK6812MINI_PLCC4_3.5x3.5mm_P1.75mm, LED_SMD:LED_SK6812MINI_PLCC4_3.5x3.5mm_P1.75mm, F.Cu at (116.8, 73.0)
- added REF**: Potentiometer_Alps_RK09L_Single_Vertical, Potentiometer_THT:Potentiometer_Alps_RK09L_Single_Vertical, F.Cu at (147.2, 138.4)
- added REF**: Potentiometer_Alps_RK09L_Single_Vertical, Potentiometer_THT:Potentiometer_Alps_RK09L_Single_Vertical, F.Cu at (172.6, 138.4)
- added REF**: CONN_MJ-3502, audioJack:CONN_MJ-3502, F.Cu at (157.4, 19.7)
- added REF**: LED_SK6812MINI_PLCC4_3.5x3.5mm_P1.75mm, LED_SMD:LED_SK6812MINI_PLCC4_3.5x3.5mm_P1.75mm, F.Cu at (116.8, 93.3)
- added REF**: Potentiometer_Alps_RK09L_Single_Vertical, Potentiometer_THT:Potentiometer_Alps_RK09L_Single_Vertical, F.Cu at (119.3, 17.1)
- added REF**: LED_SK6812MINI_PLCC4_3.5x3.5mm_P1.75mm, LED_SMD:LED_SK6812MINI_PLCC4_3.5x3.5mm_P1.75mm, F.Cu at (88.8, 92.7)
- added REF**: LED_SK6812MINI_PLCC4_3.5x3.5mm_P1.75mm, LED_SMD:LED_SK6812MINI_PLCC4_3.5x3.5mm_P1.75mm, F.Cu at (88.7, 31.8)
- moved REF** 210.0 mm to (35.4, 16.5), turned to -90 degrees
- moved REF** 196.0 mm to (-114.3, 124.5), turned to -90 degrees
- moved REF** 192.4 mm to (-110.8, 27.0), turned to 0 degrees
- moved REF** 191.4 mm to (29.1, 158.7), turned to 180 degrees
- moved REF** 183.7 mm to (35.4, 36.2), turned to -90 degrees
- moved REF** 178.0 mm to (63.4, 15.8), turned to -90 degrees
- moved REF** 160.9 mm to (35.4, 56.5), turned to -90 degrees
- moved REF** 160.8 mm to (55.8, 161.3), turned to 180 degrees
- moved ? 159.2 mm to (28.2, 127.5), turned to 180 degrees
- moved REF** 153.5 mm to (35.4, 137.8), turned to -90 degrees
- moved REF** 152.7 mm to (-101.6, 30.5), turned to 90 degrees
- moved REF** 152.5 mm to (63.4, 36.2), turned to -90 degrees
- moved REF** 145.2 mm to (91.4, 16.5), turned to -90 degrees
- moved REF** 144.7 mm to (35.4, 76.8), turned to -90 degrees
- moved U1 142.4 mm to (-101.6, 96.5), turned to 90 degrees
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Routing:
- net (no net): track 471.3 -> 68.6 mm
Other:
- board outline added: 1.3 x 11.1 mm
- board text added: "Potentiometer_Alps_RK09L_Single_Vertical"

Commit message: moar
booooooard
Parts:
- removed ? (x6): , 
- removed REF** (x42): LED_SK6812MINI_PLCC4_3.5x3.5mm_P1.75mm, LED_SMD:LED_SK6812MINI_PLCC4_3.5x3.5mm_P1.75mm
- removed REF** (x42): Potentiometer_Alps_RK09L_Single_Vertical, Potentiometer_THT:Potentiometer_Alps_RK09L_Single_Vertical
- removed REF** (x7): N16, cd74hc4051:N16
- removed REF** (x6): CONN_MJ-3502, audioJack:CONN_MJ-3502
- removed REF**: DQS20_TEX, txb0108dqsr:DQS20_TEX
- removed REF**: BarrelJack_Horizontal, Connector_BarrelJack:BarrelJack_Horizontal
- removed REF**: Adafruit_SSD1306, Display:Adafruit_SSD1306
- removed REF** (x2): KYCON_KCDX-5S-N, midiJack:KYCON_KCDX-5S-N
- added D1: NeoPixel_THT, LED_SMD:LED_SK6812MINI_PLCC4_3.5x3.5mm_P1.75mm, F.Cu at (182.9, 99.1)
- added D10: NeoPixel_THT, LED_SMD:LED_SK6812MINI_PLCC4_3.5x3.5mm_P1.75mm, F.Cu at (185.2, 83.9)
- added D11: NeoPixel_THT, LED_SMD:LED_SK6812MINI_PLCC4_3.5x3.5mm_P1.75mm, F.Cu at (157.6, 127.0)
- added D12: NeoPixel_THT, LED_SMD:LED_SK6812MINI_PLCC4_3.5x3.5mm_P1.75mm, F.Cu at (171.1, 110.1)
- added D13: NeoPixel_THT, LED_SMD:LED_SK6812MINI_PLCC4_3.5x3.5mm_P1.75mm, F.Cu at (81.5, 57.8)
- added D14: NeoPixel_THT, LED_SMD:LED_SK6812MINI_PLCC4_3.5x3.5mm_P1.75mm, F.Cu at (135.4, 47.9)
- added D15: NeoPixel_THT, LED_SMD:LED_SK6812MINI_PLCC4_3.5x3.5mm_P1.75mm, F.Cu at (164.1, 115.2)
- added D16: NeoPixel_THT, LED_SMD:LED_SK6812MINI_PLCC4_3.5x3.5mm_P1.75mm, F.Cu at (241.2, 34.3)
- added D17: NeoPixel_THT, LED_SMD:LED_SK6812MINI_PLCC4_3.5x3.5mm_P1.75mm, F.Cu at (216.1, 60.3)
- added D18: NeoPixel_THT, LED_SMD:LED_SK6812MINI_PLCC4_3.5x3.5mm_P1.75mm, F.Cu at (200.6, 69.6)
- added D19: NeoPixel_THT, LED_SMD:LED_SK6812MINI_PLCC4_3.5x3.5mm_P1.75mm, F.Cu at (185.2, 94.0)
- added D2: NeoPixel_THT, LED_SMD:LED_SK6812MINI_PLCC4_3.5x3.5mm_P1.75mm, F.Cu at (175.9, 98.3)
- added D20: NeoPixel_THT, LED_SMD:LED_SK6812MINI_PLCC4_3.5x3.5mm_P1.75mm, F.Cu at (225.7, 48.6)
- added D21: NeoPixel_THT, LED_SMD:LED_SK6812MINI_PLCC4_3.5x3.5mm_P1.75mm, F.Cu at (185.2, 89.0)
- added D22: NeoPixel_THT, LED_SMD:LED_SK6812MINI_PLCC4_3.5x3.5mm_P1.75mm, F.Cu at (230.1, 53.7)
- added D23: NeoPixel_THT, LED_SMD:LED_SK6812MINI_PLCC4_3.5x3.5mm_P1.75mm, F.Cu at (200.6, 79.7)
- added D24: NeoPixel_THT, LED_SMD:LED_SK6812MINI_PLCC4_3.5x3.5mm_P1.75mm, F.Cu at (81.5, 47.7)
- added D25: NeoPixel_THT, LED_SMD:LED_SK6812MINI_PLCC4_3.5x3.5mm_P1.75mm, F.Cu at (250.9, 31.6)
- added D26: NeoPixel_THT, LED_SMD:LED_SK6812MINI_PLCC4_3.5x3.5mm_P1.75mm, F.Cu at (223.1, 60.3)
- added D27: NeoPixel_THT, LED_SMD:LED_SK6812MINI_PLCC4_3.5x3.5mm_P1.75mm, F.Cu at (235.5, 40.9)
- added D28: NeoPixel_THT, LED_SMD:LED_SK6812MINI_PLCC4_3.5x3.5mm_P1.75mm, F.Cu at (207.7, 74.6)
- added D29: NeoPixel_THT, LED_SMD:LED_SK6812MINI_PLCC4_3.5x3.5mm_P1.75mm, F.Cu at (242.5, 39.3)
- added D3: NeoPixel_THT, LED_SMD:LED_SK6812MINI_PLCC4_3.5x3.5mm_P1.75mm, F.Cu at (250.9, 26.5)
- added D30: NeoPixel_THT, LED_SMD:LED_SK6812MINI_PLCC4_3.5x3.5mm_P1.75mm, F.Cu at (164.1, 110.1)
- added D31: NeoPixel_THT, LED_SMD:LED_SK6812MINI_PLCC4_3.5x3.5mm_P1.75mm, F.Cu at (81.5, 52.7)
- added D32: NeoPixel_THT, LED_SMD:LED_SK6812MINI_PLCC4_3.5x3.5mm_P1.75mm, F.Cu at (175.9, 103.3)
- added D33: NeoPixel_THT, LED_SMD:LED_SK6812MINI_PLCC4_3.5x3.5mm_P1.75mm, F.Cu at (235.5, 45.9)
- added D34: NeoPixel_THT, LED_SMD:LED_SK6812MINI_PLCC4_3.5x3.5mm_P1.75mm, F.Cu at (199.2, 84.7)
- added D35: NeoPixel_THT, LED_SMD:LED_SK6812MINI_PLCC4_3.5x3.5mm_P1.75mm, F.Cu at (200.6, 74.6)
- added D36: NeoPixel_THT, LED_SMD:LED_SK6812MINI_PLCC4_3.5x3.5mm_P1.75mm, F.Cu at (216.1, 65.3)
- added D37: NeoPixel_THT, LED_SMD:LED_SK6812MINI_PLCC4_3.5x3.5mm_P1.75mm, F.Cu at (207.7, 69.6)
- added D38: NeoPixel_THT, LED_SMD:LED_SK6812MINI_PLCC4_3.5x3.5mm_P1.75mm, F.Cu at (223.1, 55.2)
- added D39: NeoPixel_THT, LED_SMD:LED_SK6812MINI_PLCC4_3.5x3.5mm_P1.75mm, F.Cu at (130.4, 90.9)
- added D4: NeoPixel_THT, LED_SMD:LED_SK6812MINI_PLCC4_3.5x3.5mm_P1.75mm, F.Cu at (216.1, 55.2)
- added D40: NeoPixel_THT, LED_SMD:LED_SK6812MINI_PLCC4_3.5x3.5mm_P1.75mm, F.Cu at (164.1, 120.2)
- added D41: NeoPixel_THT, LED_SMD:LED_SK6812MINI_PLCC4_3.5x3.5mm_P1.75mm, F.Cu at (150.6, 127.0)
- added D42: NeoPixel_THT, LED_SMD:LED_SK6812MINI_PLCC4_3.5x3.5mm_P1.75mm, F.Cu at (192.2, 83.9)
- added D43: 1N4148, Diode_THT:D_DO-35_SOD27_P7.62mm_Horizontal, F.Cu at (79.6, 43.4)
- added D5: NeoPixel_THT, LED_SMD:LED_SK6812MINI_PLCC4_3.5x3.5mm_P1.75mm, F.Cu at (123.4, 90.9)
- added D6: NeoPixel_THT, LED_SMD:LED_SK6812MINI_PLCC4_3.5x3.5mm_P1.75mm, F.Cu at (140.8, 139.8)
- added D7: NeoPixel_THT, LED_SMD:LED_SK6812MINI_PLCC4_3.5x3.5mm_P1.75mm, F.Cu at (192.2, 89.0)
- added D8: NeoPixel_THT, LED_SMD:LED_SK6812MINI_PLCC4_3.5x3.5mm_P1.75mm, F.Cu at (140.8, 134.7)
- added D9: NeoPixel_THT, LED_SMD:LED_SK6812MINI_PLCC4_3.5x3.5mm_P1.75mm, F.Cu at (147.9, 134.7)
- added J1: Barrel_Jack, Connector_BarrelJack:BarrelJack_CUI_PJ-102AH_Horizontal, F.Cu at (91.6, 89.2)
- added J2: MIDI OUT, midiJack:KYCON_KCDX-5S-N, F.Cu at (79.9, 33.1)
- added J3: MIDI IN, midiJack:KYCON_KCDX-5S-N, F.Cu at (60.5, 108.0)
- added J4: MJ-3502, audioJack:CONN_MJ-3502, F.Cu at (78.8, 111.5)
- added J5: MJ-3502, audioJack:CONN_MJ-3502, F.Cu at (111.8, 57.9)
- added J6: MJ-3502, audioJack:CONN_MJ-3502, F.Cu at (140.4, 36.6)
- added J7: MJ-3502, audioJack:CONN_MJ-3502, F.Cu at (73.4, 54.2)
- added J8: MJ-3502, audioJack:CONN_MJ-3502, F.Cu at (90.7, 79.3)
- added J9: MJ-3502, audioJack:CONN_MJ-3502, F.Cu at (99.8, 79.3)
- added OLED1: OLED1.3, Display:Adafruit_SSD1306, F.Cu at (58.9, 65.6)
- added R1: 220R, Resistor_THT:R_Axial_DIN0204_L3.6mm_D1.6mm_P2.54mm_Vertical, F.Cu at (100.2, 91.6)
- added R10: R_Potentiometer, Potentiometer_THT:Potentiometer_Alps_RK09K_Single_Vertical, F.Cu at (131.4, 100.4)
- added R11: R_Potentiometer, Potentiometer_THT:Potentiometer_Alps_RK09K_Single_Vertical, F.Cu at (208.4, 28.7)
- added R12: R_Potentiometer, Potentiometer_THT:Potentiometer_Alps_RK09K_Single_Vertical, F.Cu at (137.0, 71.7)
- added R13: R_Potentiometer, Potentiometer_THT:Potentiometer_Alps_RK09K_Single_Vertical, F.Cu at (208.4, 43.0)
- added R14: R_Potentiometer, Potentiometer_THT:Potentiometer_Alps_RK09K_Single_Vertical, F.Cu at (85.0, 108.6)
- added R15: R_Potentiometer, Potentiometer_THT:Potentiometer_Alps_RK09K_Single_Vertical, F.Cu at (118.1, 50.0)
- added R16: R_Potentiometer, Potentiometer_THT:Potentiometer_Alps_RK09K_Single_Vertical, F.Cu at (183.3, 57.4)
- added R17: R_Potentiometer, Potentiometer_THT:Potentiometer_Alps_RK09K_Single_Vertical, F.Cu at (115.9, 100.0)
- added R18: R_Potentiometer, Potentiometer_THT:Potentiometer_Alps_RK09K_Single_Vertical, F.Cu at (193.0, 28.7)
- added R19: R_Potentiometer, Potentiometer_THT:Potentiometer_Alps_RK09K_Single_Vertical, F.Cu at (167.9, 86.1)
- added R2: 220R, Resistor_THT:R_Axial_DIN0204_L3.6mm_D1.6mm_P2.54mm_Vertical, F.Cu at (140.5, 45.7)
- added R20: R_Potentiometer, Potentiometer_THT:Potentiometer_Alps_RK09K_Single_Vertical, F.Cu at (167.9, 57.4)
- added R21: R_Potentiometer, Potentiometer_THT:Potentiometer_Alps_RK09K_Single_Vertical, F.Cu at (183.3, 71.7)
- added R22: R_Potentiometer, Potentiometer_THT:Potentiometer_Alps_RK09K_Single_Vertical, F.Cu at (61.8, 123.8)
- added R23: R_Potentiometer, Potentiometer_THT:Potentiometer_Alps_RK09K_Single_Vertical, F.Cu at (167.9, 71.7)
- added R24: R_Potentiometer, Potentiometer_THT:Potentiometer_Alps_RK09K_Single_Vertical, F.Cu at (92.7, 128.7)
- added R25: R_Potentiometer, Potentiometer_THT:Potentiometer_Alps_RK09K_Single_Vertical, F.Cu at (152.4, 86.1)
- added R26: R_Potentiometer, Potentiometer_THT:Potentiometer_Alps_RK09K_Single_Vertical, F.Cu at (146.8, 114.8)
- added R27: R_Potentiometer, Potentiometer_THT:Potentiometer_Alps_RK09K_Single_Vertical, F.Cu at (100.5, 114.4)
- added R28: R_Potentiometer, Potentiometer_THT:Potentiometer_Alps_RK09K_Single_Vertical, F.Cu at (100.5, 100.0)
- added R29: R_Potentiometer, Potentiometer_THT:Potentiometer_Alps_RK09K_Single_Vertical, F.Cu at (146.6, 28.7)
- added R3: 220R, Resistor_THT:R_Axial_DIN0204_L3.6mm_D1.6mm_P2.54mm_Vertical, F.Cu at (51.1, 139.4)
- added R30: R_Potentiometer, Potentiometer_THT:Potentiometer_Alps_RK09K_Single_Vertical, F.Cu at (106.1, 71.3)
- added R31: R_Potentiometer, Potentiometer_THT:Potentiometer_Alps_RK09K_Single_Vertical, F.Cu at (152.4, 71.7)
- added R32: R_Potentiometer, Potentiometer_THT:Potentiometer_Alps_RK09K_Single_Vertical, F.Cu at (108.1, 128.7)
- added R33: R_Potentiometer, Potentiometer_THT:Potentiometer_Alps_RK09K_Single_Vertical, F.Cu at (223.9, 28.7)
- added R34: R_Potentiometer, Potentiometer_THT:Potentiometer_Alps_RK09K_Single_Vertical, F.Cu at (177.5, 28.7)
- added R35: R_Potentiometer, Potentiometer_THT:Potentiometer_Alps_RK09K_Single_Vertical, F.Cu at (77.2, 123.8)
- added R36: R_Potentiometer, Potentiometer_THT:Potentiometer_Alps_RK09K_Single_Vertical, F.Cu at (198.8, 57.4)
- added R37: R_Potentiometer, Potentiometer_THT:Potentiometer_Alps_RK09K_Single_Vertical, F.Cu at (137.0, 86.1)
- added R38: R_Potentiometer, Potentiometer_THT:Potentiometer_Alps_RK09K_Single_Vertical, F.Cu at (162.1, 28.7)
- added R39: R_Potentiometer, Potentiometer_THT:Potentiometer_Alps_RK09K_Single_Vertical, F.Cu at (152.4, 57.4)
- added R4: 220R, Resistor_THT:R_Axial_DIN0204_L3.6mm_D1.6mm_P2.54mm_Vertical, F.Cu at (100.2, 88.4)
- added R40: R_Potentiometer, Potentiometer_THT:Potentiometer_Alps_RK09K_Single_Vertical, F.Cu at (193.0, 43.0)
- added R41: R_Potentiometer, Potentiometer_THT:Potentiometer_Alps_RK09K_Single_Vertical, F.Cu at (115.9, 114.4)
- added R42: R_Potentiometer, Potentiometer_THT:Potentiometer_Alps_RK09K_Single_Vertical, F.Cu at (123.6, 129.1)
- added R43: R_Potentiometer, Potentiometer_THT:Potentiometer_Alps_RK09K_Single_Vertical, F.Cu at (162.1, 43.0)
- added R44: R_Potentiometer, Potentiometer_THT:Potentiometer_Alps_RK09K_Single_Vertical, F.Cu at (146.6, 43.0)
- added R45: R_Potentiometer, Potentiometer_THT:Potentiometer_Alps_RK09K_Single_Vertical, F.Cu at (131.4, 114.8)
- added R46: R_Potentiometer, Potentiometer_THT:Potentiometer_Alps_RK09K_Single_Vertical, F.Cu at (121.5, 78.7)
- added R5: R_Potentiometer, Potentiometer_THT:Potentiometer_Alps_RK09K_Single_Vertical, F.Cu at (137.0, 57.4)
- added R6: R_Potentiometer, Potentiometer_THT:Potentiometer_Alps_RK09K_Single_Vertical, F.Cu at (121.5, 64.3)
- added R7: R_Potentiometer, Potentiometer_THT:Potentiometer_Alps_RK09K_Single_Vertical, F.Cu at (106.1, 85.7)
- added R8: R_Potentiometer, Potentiometer_THT:Potentiometer_Alps_RK09K_Single_Vertical, F.Cu at (177.5, 43.0)
- added R9: R_Potentiometer, Potentiometer_THT:Potentiometer_Alps_RK09K_Single_Vertical, F.Cu at (146.8, 100.4)
- added S1: B3F-4055, Button_Switch_THT:SW_TH_Tactile_Omron_B3F-10xx, F.Cu at (81.2, 135.1)
- added S2: B3F-4055, Button_Switch_THT:SW_TH_Tactile_Omron_B3F-10xx, F.Cu at (239.3, 25.6)
- added S3: B3F-4055, Button_Switch_THT:SW_TH_Tactile_Omron_B3F-10xx, F.Cu at (139.0, 126.1)
- added S4: B3F-4055, Button_Switch_THT:SW_TH_Tactile_Omron_B3F-10xx, F.Cu at (223.8, 40.0)
- added S5: B3F-4055, Button_Switch_THT:SW_TH_Tactile_Omron_B3F-10xx, F.Cu at (71.5, 135.1)
- added S6: B3F-4055, Button_Switch_THT:SW_TH_Tactile_Omron_B3F-10xx, F.Cu at (61.7, 135.1)
- added U10: 6N138, Package_DIP:DIP-8_W7.62mm_Socket, F.Cu at (162.7, 97.9)
- added U2: TXB0108DQSR, Package_SON:USON-20_2x4mm_P0.4mm, F.Cu at (256.6, 26.8)
- added U3: 74HC4051, cd74hc4051:N16, F.Cu at (113.2, 43.5)
- added U4: 74HC4051, cd74hc4051:N16, F.Cu at (102.6, 43.5)
- added U5: 74HC4051, cd74hc4051:N16, F.Cu at (134.3, 43.5)
- added U6: 74HC4051, cd74hc4051:N16, F.Cu at (58.6, 136.1)
- added U7: 74HC4051, cd74hc4051:N16, F.Cu at (95.2, 64.9)
- added U8: 74HC4051, cd74hc4051:N16, F.Cu at (123.8, 43.5)
- added U9: 74HC4051, cd74hc4051:N16, F.Cu at (105.8, 64.9)
- U1: value Teensy4.0 -> teensy 4.0
- moved U1 169.4 mm to (59.2, 43.2), turned to 0 degrees
Connections:
- U1 pad 0: (no net) -> MIDI IN
- U1 pad 1: (no net) -> MIDI OUT
- U1 pad 10: (no net) -> M4
- U1 pad 11: (no net) -> M5
- U1 pad 12: (no net) -> M6
- U1 pad 13: (no net) -> unconnected-(U1-Pad13)
- U1 pad 14: (no net) -> A0
- U1 pad 15: (no net) -> A1
- U1 pad 16: (no net) -> A2
- U1 pad 17: (no net) -> A3
- U1 pad 18: (no net) -> SDA
- U1 pad 19: (no net) -> SCL
- U1 pad 2: (no net) -> unconnected-(U1-Pad2)
- U1 pad 20: (no net) -> A4
- U1 pad 21: (no net) -> A5
- U1 pad 22: (no net) -> MUX_READ
- U1 pad 23: (no net) -> unconnected-(U1-Pad23)
- U1 pad 3: (no net) -> unconnected-(U1-Pad3)
- U1 pad 3.3V_1: (no net) -> unconnected-(U1-Pad3.3V_1)
- U1 pad 3.3V_2: (no net) -> Net-(U1-Pad3.3V_2)
- U1 pad 4: (no net) -> unconnected-(U1-Pad4)
- U1 pad 5: (no net) -> unconnected-(U1-Pad5)
- U1 pad 6: (no net) -> LED
- U1 pad 7: (no net) -> M1
- U1 pad 8: (no net) -> M2
- U1 pad 9: (no net) -> M3
- U1 pad G1: (no net) -> GROUND
- U1 pad G2: (no net) -> GROUND
- U1 pad G3: (no net) -> unconnected-(U1-PadG3)
- U1 pad ON-OFF: (no net) -> unconnected-(U1-PadON-OFF)
- U1 pad PGM: (no net) -> unconnected-(U1-PadPGM)
- U1 pad VBAT: (no net) -> unconnected-(U1-PadVBAT)
- U1 pad VIN: (no net) -> 5VDC
Routing:
- net (no net): track 68.6 -> 0.00 mm
Other:
- board text removed: "Potentiometer_Alps_RK09L_Single_Vertical"

Commit message: board
moar
Parts:
- removed OLED1: OLED1.3, Display:Adafruit_SSD1306
- removed S1, S2, S3, S4, S5, S6: B3F-4055, Button_Switch_THT:SW_TH_Tactile_Omron_B3F-10xx
- added J10: I2C_STANDARDJS-1MM, Connector_JST:JST_EH_S4B-EH_1x04_P2.50mm_Horizontal, F.Cu at (102.9, 38.1)
- added SW1: SW_MEC_5E, Button_Switch_THT:SW_TH_Tactile_Omron_B3F-10xx, F.Cu at (98.3, 167.9)
- added SW2: SW_MEC_5E, Button_Switch_THT:SW_TH_Tactile_Omron_B3F-10xx, F.Cu at (83.1, 167.9)
- added SW3: SW_MEC_5E, Button_Switch_THT:SW_TH_Tactile_Omron_B3F-10xx, F.Cu at (111.0, 162.8)
- added SW4: SW_MEC_5E, Button_Switch_THT:SW_TH_Tactile_Omron_B3F-10xx, F.Cu at (111.0, 175.6)
- added SW5: SW_MEC_5E, Button_Switch_THT:SW_TH_Tactile_Omron_B3F-10xx, F.Cu at (67.9, 167.9)
- added SW6: SW_MEC_5E, Button_Switch_THT:SW_TH_Tactile_Omron_B3F-10xx, F.Cu at (85.7, 180.6)
- moved U2 167.1 mm to (154.9, 159.4), turned to 180 degrees
- moved U1 162.0 mm to (185.4, 144.8)
- moved D31 158.8 mm to (240.1, 45.0)
- moved U3 155.9 mm to (43.2, 182.9)
- moved R43 155.2 mm to (45.3, 145.2)
- moved D16 143.7 mm to (139.8, 136.1)
- moved R13 135.7 mm to (86.7, 103.0)
- moved R40 129.7 mm to (107.1, 140.2)
- moved D35 125.8 mm to (101.8, 152.4)
- moved D3 123.6 mm to (166.5, 116.7)
- moved R30 119.2 mm to (222.8, 47.1)
- moved D10 119.1 mm to (87.7, 152.4)
- moved D20 115.5 mm to (144.8, 131.1)
- moved R29 113.0 mm to (122.5, 139.0)
- moved D43 112.6 mm to (60.6, 154.3)
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Connections:
- U1 pad G3: unconnected-(U1-PadG3) -> GROUND

Commit message: circuit/board
finalizing power regulation
Parts:
- added C1: CAP_CERAMIC0402, Capacitor_THT:C_Disc_D4.3mm_W1.9mm_P5.00mm, F.Cu at (215.9, 111.8)
- added C2: CAP_CERAMIC0402, Capacitor_THT:C_Disc_D4.3mm_W1.9mm_P5.00mm, F.Cu at (229.3, 105.2)
- added D44: 1N4007, Diode_THT:D_DO-41_SOD81_P10.16mm_Horizontal, F.Cu at (204.7, 105.6)
- added SW7: SW_Push_SPDT, Button_Switch_THT:SW_PUSH_6mm, F.Cu at (204.8, 115.7)
- added TH1: Thermistor, Capacitor_THT:C_Disc_D9.0mm_W5.0mm_P7.50mm, F.Cu at (218.5, 106.8)
- added U11: LM317_TO-220, Package_TO_SOT_THT:TO-220-3_Vertical, F.Cu at (206.0, 111.7)
Connections:
- J1 pad 1: 5VDC -> +5V
- U1 pad VIN: 5VDC -> Net-(U1-PadVIN)
- U2 pad 16: 5VDC -> Net-(U1-PadVIN)

Commit message: kicad again
might need to restart layout
Parts:
- moved R11 222.3 mm to (29.5, 180.4)
- moved J3 206.7 mm to (226.1, 68.6), turned to 90 degrees
- moved J2 200.5 mm to (218.4, 43.2), turned to 90 degrees
- moved J9 195.2 mm to (172.7, 180.3), turned to 180 degrees
- moved J1 187.5 mm to (196.3, 39.2), turned to 180 degrees
- moved D1 176.7 mm to (35.6, 50.8)
- moved J4 172.7 mm to (142.2, 180.3), turned to 180 degrees
- moved D43 164.8 mm to (207.0, 78.7)
- moved R16 161.2 mm to (60.0, 139.7)
- moved J5 157.7 mm to (111.8, 180.3), turned to 180 degrees
- moved J6 157.7 mm to (50.8, 180.3), turned to 180 degrees
- moved J7 153.7 mm to (20.3, 180.3), turned to 180 degrees
- moved D2 153.5 mm to (35.6, 71.1)
- moved D8 153.3 mm to (66.0, 50.8)
- moved J8 152.4 mm to (81.3, 180.3), turned to 180 degrees
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Connections:
- net Net-(U2-Pad17) renamed MuxA3
- net Net-(U2-Pad18) renamed MuxA2
- net Net-(U2-Pad19) renamed MuxA1
- net Net-(U2-Pad20) renamed MUX_OUT
- net Net-(U3-Pad1) renamed MuxBD5
- net Net-(U3-Pad12) renamed MuxBD4
- net Net-(U3-Pad13) renamed MuxBD1
- net Net-(U3-Pad14) renamed MuxBD2
- net Net-(U3-Pad15) renamed MuxBD3
- net Net-(U3-Pad5) renamed MuxBD6
- SW1 pad 2: unconnected-(SW1-Pad2) -> 5VDC
- SW2 pad 2: unconnected-(SW2-Pad2) -> 5VDC
- SW3 pad 2: unconnected-(SW3-Pad2) -> 5VDC
- SW4 pad 2: unconnected-(SW4-Pad2) -> 5VDC
- SW5 pad 2: unconnected-(SW5-Pad2) -> 5VDC
- SW6 pad 2: unconnected-(SW6-Pad2) -> 5VDC
- TH1 pad 1: unconnected-(TH1-Pad1) -> 5VDC
Routing:
- net GROUND: track 0.00 -> 1236.0 mm
- net 5VDC: track 0.00 -> 206.2 mm
- net B4_2: track 0.00 -> 24.7 mm
- net Net-(D44-Pad1): track 0.00 -> 17.9 mm
- net Net-(D43-Pad2): track 0.00 -> 17.5 mm
- net Net-(SW7-Pad2): track 0.00 -> 16.5 mm
- net Net-(D43-Pad1): track 0.00 -> 15.3 mm
- net Net-(J2-Pad5): track 0.00 -> 13.7 mm
- net Net-(U1-PadVIN): track 0.00 -> 9.20 mm
- net B4_1: track 0.00 -> 6.96 mm
- net Net-(D44-Pad2): track 0.00 -> 5.66 mm
- net MIDI IN: track 0.00 -> 5.39 mm
- net Net-(J3-Pad4): track 0.00 -> 3.93 mm
Other:
- outline, holes or cut-outs redrawn

Commit message: two boards one git
two boards now - one for ui, the other for ics and io
Parts:
- removed D1, D10, D11, D12, D13, D14, D15, D16, D17, D18, D19, D2, D20, D21, D22, D23, D24, D25, D26, D27, D28, D29, D3, D30, D31, D32, D33, D34, D35, D36, D37, D38, D39, D4, D40, D41, D42, D5, D6, D7, D8, D9: NeoPixel_THT, LED_SMD:LED_SK6812MINI_PLCC4_3.5x3.5mm_P1.75mm
- removed R10, R11, R12, R13, R14, R15, R16, R17, R18, R19, R20, R21, R22, R23, R24, R25, R26, R27, R28, R29, R30, R31, R32, R33, R34, R35, R36, R37, R38, R39, R40, R41, R42, R43, R44, R45, R46, R5, R6, R7, R8, R9: R_Potentiometer, Potentiometer_THT:Potentiometer_Alps_RK09K_Single_Vertical
- removed SW1, SW2, SW3, SW4, SW5, SW6: SW_MEC_5E, Button_Switch_THT:SW_TH_Tactile_Omron_B3F-10xx
- added J11: Conn_01x02, Connector_PinHeader_1.00mm:PinHeader_1x02_P1.00mm_Vertical, F.Cu at (134.6, 38.1)
- added J12: Conn_01x07, Connector_PinHeader_1.00mm:PinHeader_1x07_P1.00mm_Vertical, F.Cu at (134.6, 29.1)
- added J13: Conn_01x07, Connector_PinHeader_1.00mm:PinHeader_1x07_P1.00mm_Vertical, F.Cu at (151.4, 29.1)
- added J14: Conn_01x07, Connector_PinHeader_1.00mm:PinHeader_1x07_P1.00mm_Vertical, F.Cu at (144.7, 29.1)
- added J15: Conn_01x07, Connector_PinHeader_1.00mm:PinHeader_1x07_P1.00mm_Vertical, F.Cu at (148.0, 29.1)
- added J16: Conn_01x07, Connector_PinHeader_1.00mm:PinHeader_1x07_P1.00mm_Vertical, F.Cu at (138.0, 29.1)
- added J17: Conn_01x07, Connector_PinHeader_1.00mm:PinHeader_1x07_P1.00mm_Vertical, F.Cu at (141.3, 29.1)
- added J18: Conn_01x07, Connector_PinHeader_1.00mm:PinHeader_1x07_P1.00mm_Vertical, F.Cu at (154.7, 29.1)
- added U12: CD74HC4050E, cd74hc4051:N16, F.Cu at (69.8, 72.4)
- U2: value TXB0108DQSR -> CD74HC4050E; footprint Package_SON:USON-20_2x4mm_P0.4mm -> cd74hc4051:N16
- moved J3 203.3 mm to (27.9, 22.9), turned to 180 degrees
- moved U9 189.0 mm to (-12.2, 84.7)
- moved R1 186.5 mm to (30.5, 45.7), turned to 0 degrees
- moved D43 177.8 mm to (33.0, 41.9), turned to 90 degrees
- moved U10 174.4 mm to (39.4, 34.3), turned to 0 degrees
- moved R2 161.3 mm to (35.6, 50.8), turned to -90 degrees
- moved J2 158.8 mm to (61.0, 22.9), turned to 180 degrees
- moved U8 143.5 mm to (3.05, 62.7)
- moved R4 129.0 mm to (73.7, 35.6), turned to 180 degrees
- moved U7 128.3 mm to (-12.2, 62.7)
- moved R3 124.6 mm to (53.3, 38.1)
- moved J4 123.4 mm to (27.6, 134.6)
- moved U2 114.9 mm to (8.89, 85.1)
- moved C1 114.6 mm to (68.6, 35.6), turned to 180 degrees
- moved J1 110.5 mm to (86.4, 27.9)
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Connections:
- U1 pad 3.3V_2: Net-(U1-Pad3.3V_2) -> 3VDC
- U2 pad 1: MUX_READ -> 5VDC
- U2 pad 10: LED -> MuxB1
- U2 pad 11: LED_CNTRL -> M5
- U2 pad 12: MuxB3 -> MuxB2
- U2 pad 13: MuxB2 -> unconnected-(U2-Pad13)
- U2 pad 14: MuxB1 -> M6
- U2 pad 15: GROUND -> MuxB3
- U2 pad 16: Net-(U1-PadVIN) -> unconnected-(U2-Pad16)
- U2 pad 2: M1 -> MuxA1
- U2 pad 3: M2 -> M1
- U2 pad 4: M3 -> MuxA2
- U2 pad 5: Net-(U1-Pad3.3V_2) -> M2
- U2 pad 6: unconnected-(U2-Pad6) -> MuxA3
- U2 pad 7: M4 -> M3
- U2 pad 8: M5 -> GROUND
- U2 pad 9: M6 -> M4
Routing:
- net GROUND: track 1236.0 -> 114.3 mm
- net 5VDC: track 206.2 -> 72.6 mm
- net MuxBD1: track 0.00 -> 83.0 mm
- net Net-(U1-PadVIN): track 9.20 -> 68.9 mm
- net MuxBD3: track 0.00 -> 50.4 mm
- net Net-(C1-Pad1): track 17.9 -> 67.7 mm
- net M4: track 0.00 -> 33.9 mm
- net M3: track 0.00 -> 30.0 mm
- net M5: track 0.00 -> 27.7 mm
- net M1: track 0.00 -> 27.0 mm
- net M2: track 0.00 -> 25.2 mm
- net B4_2: track 24.7 -> 0.00 mm
- net MIDI IN: track 5.39 -> 28.1 mm
- net MIDI OUT: track 0.00 -> 21.8 mm
- net M6: track 0.00 -> 19.9 mm
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