File: BenzKnobz/BenzKnobz.kicad_pcb (KiCad board)
At the start: 2 copper layers, 1.3 x 11.1 mm, 40 parts, among them J1 Barrel_Jack, J10 I2C_STANDARDJS-1MM, J11 Conn_01x02, J12 Conn_01x07, J13 Conn_01x07, J14 Conn_01x07, J15 Conn_01x07, J16 Conn_01x07, J17 Conn_01x07, J18 Conn_01x07, J2 MIDI OUT, J3 MIDI IN, J4 MJ-3502, J5 MJ-3502, J6 MJ-3502, J7 MJ-3502, J8 MJ-3502, J9 MJ-3502, SW7 SW_Push_SPDT, U1 teensy 4.0, U10 6N138, U11 LM317_TO-220, U12 CD74HC4050E, U2 CD74HC4050E, U3 74HC4051, U4 74HC4051, U5 74HC4051, U6 74HC4051, U7 74HC4051, U8 74HC4051, U9 74HC4051

Commit message: brd
moar - almost completely laid out
Parts:
- removed J18: Conn_01x07, Connector_PinHeader_1.00mm:PinHeader_1x07_P1.00mm_Vertical
- J10: value I2C_STANDARDJS-1MM -> Conn_01x03; footprint Connector_JST:JST_EH_S4B-EH_1x04_P2.50mm_Horizontal -> Connector_PinHeader_1.00mm:PinHeader_1x03_P1.00mm_Vertical
- J11: value Conn_01x02 -> Conn_01x03; footprint Connector_PinHeader_1.00mm:PinHeader_1x02_P1.00mm_Vertical -> Connector_PinHeader_1.00mm:PinHeader_1x03_P1.00mm_Vertical
- J12, J13, J14, J15, J16, J17: value Conn_01x07 -> Conn_02x04_Odd_Even_Shielded; footprint Connector_PinHeader_1.00mm:PinHeader_1x07_P1.00mm_Vertical -> Connector_PinHeader_1.00mm:PinHeader_2x04_P1.00mm_Vertical
- moved J5 141.4 mm to (149.6, 39.0), turned to 0 degrees
- moved J7 128.5 mm to (140.4, 39.0), turned to 0 degrees
- moved U7 126.5 mm to (113.2, 46.0)
- moved J4 125.6 mm to (128.8, 60.3), turned to 0 degrees
- moved U8 121.9 mm to (123.8, 46.0)
- moved U4 115.0 mm to (102.6, 46.0)
- moved U6 105.3 mm to (104.5, 67.3)
- moved J8 104.7 mm to (110.5, 60.3), turned to 0 degrees
- moved U10 99.6 mm to (137.9, 48.7)
- moved U9 95.5 mm to (83.3, 84.9)
- moved J6 92.5 mm to (119.7, 60.3), turned to 0 degrees
- moved D44 91.6 mm to (51.4, 83.9), turned to 0 degrees
- moved U5 90.1 mm to (93.9, 88.6)
- moved J15 88.7 mm to (82.0, 88.2)
- moved U2 86.8 mm to (93.9, 67.3), turned to 0 degrees
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Connections:
- J10 pad 1: GROUND -> SCL
- J10 pad 2: 5VDC -> SDA
- J10 pad 3: SDA -> LED
- J11 pad 1: 5VDC -> 3VDC
- J12 pad 1: unconnected-(J12-Pad1) -> B1_1
- J12 pad 2: unconnected-(J12-Pad2) -> B1_2
- J12 pad 3: unconnected-(J12-Pad3) -> B1_3
- J12 pad 4: unconnected-(J12-Pad4) -> B1_4
- J12 pad 5: unconnected-(J12-Pad5) -> B1_5
- J12 pad 6: unconnected-(J12-Pad6) -> B1_6
- J12 pad 7: unconnected-(J12-Pad7) -> B1_7
- J13 pad 1: unconnected-(J13-Pad1) -> B2_1
- J13 pad 2: unconnected-(J13-Pad2) -> B2_2
- J13 pad 3: unconnected-(J13-Pad3) -> B2_3
- J13 pad 4: unconnected-(J13-Pad4) -> B2_4
- J13 pad 5: unconnected-(J13-Pad5) -> B2_5
- J13 pad 6: unconnected-(J13-Pad6) -> B2_6
- J13 pad 7: unconnected-(J13-Pad7) -> B2_7
- J14 pad 1: unconnected-(J14-Pad1) -> B3_1
- J14 pad 2: unconnected-(J14-Pad2) -> B3_2
- J14 pad 3: unconnected-(J14-Pad3) -> B3_3
- J14 pad 4: unconnected-(J14-Pad4) -> B3_4
- J14 pad 5: unconnected-(J14-Pad5) -> B3_5
- J14 pad 6: unconnected-(J14-Pad6) -> B3_6
- J14 pad 7: unconnected-(J14-Pad7) -> B3_7
- J15 pad 1: unconnected-(J15-Pad1) -> B4_1
- J15 pad 2: unconnected-(J15-Pad2) -> B4_2
- J15 pad 3: unconnected-(J15-Pad3) -> B4_3
- J15 pad 4: unconnected-(J15-Pad4) -> B4_4
- J15 pad 5: unconnected-(J15-Pad5) -> B4_5
- J15 pad 6: unconnected-(J15-Pad6) -> B4_6
- J15 pad 7: unconnected-(J15-Pad7) -> B4_7
- J16 pad 1: unconnected-(J16-Pad1) -> B5_1
- J16 pad 2: unconnected-(J16-Pad2) -> B5_2
- J16 pad 3: unconnected-(J16-Pad3) -> B5_3
- J16 pad 4: unconnected-(J16-Pad4) -> B5_4
- J16 pad 5: unconnected-(J16-Pad5) -> B5_5
- J16 pad 6: unconnected-(J16-Pad6) -> B5_6
- J16 pad 7: unconnected-(J16-Pad7) -> B5_7
- J17 pad 1: unconnected-(J17-Pad1) -> B6_1
- J17 pad 2: unconnected-(J17-Pad2) -> B6_2
- J17 pad 3: unconnected-(J17-Pad3) -> B6_3
- J17 pad 4: unconnected-(J17-Pad4) -> B6_4
- J17 pad 5: unconnected-(J17-Pad5) -> B6_5
- J17 pad 6: unconnected-(J17-Pad6) -> B6_6
- J17 pad 7: unconnected-(J17-Pad7) -> B6_7
- U12 pad 10: unconnected-(U12-Pad10) -> MUX_READ
- U12 pad 11: unconnected-(U12-Pad11) -> MuxBD5
- U12 pad 12: unconnected-(U12-Pad12) -> MUX_READ
- U12 pad 14: unconnected-(U12-Pad14) -> MuxBD6
- U12 pad 15: unconnected-(U12-Pad15) -> MUX_READ
- U12 pad 3: MUX_OUT -> MuxBD1
- U12 pad 4: unconnected-(U12-Pad4) -> MUX_READ
- U12 pad 5: unconnected-(U12-Pad5) -> MuxBD2
- U12 pad 6: unconnected-(U12-Pad6) -> MUX_READ
- U12 pad 7: unconnected-(U12-Pad7) -> MuxBD3
- U12 pad 9: unconnected-(U12-Pad9) -> MuxBD4
- U8 pad 3: MuxBD6 -> MuxBD5
- U9 pad 3: MuxBD5 -> MuxBD6
Routing:
- net GROUND: track 114.3 -> 0.00 mm
- net MuxBD1: track 83.0 -> 0.00 mm
- net 5VDC: track 72.6 -> 0.00 mm
- net Net-(U1-PadVIN): track 68.9 -> 0.00 mm
- net Net-(C1-Pad1): track 67.7 -> 0.00 mm
- net MuxBD3: track 50.4 -> 0.00 mm
- net M4: track 33.9 -> 0.00 mm
- net M3: track 30.0 -> 0.00 mm
- net MIDI IN: track 28.1 -> 0.00 mm
- net M5: track 27.7 -> 0.00 mm
- net M1: track 27.0 -> 0.00 mm
- net M2: track 25.2 -> 0.00 mm
- net MIDI OUT: track 21.8 -> 0.00 mm
- net M6: track 19.9 -> 0.00 mm
- net Net-(J3-Pad4): track 18.7 -> 0.00 mm
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Other:
- outline, holes or cut-outs redrawn
