File: BenzKnobz/BenzKnobz.kicad_sch (KiCad schematic)
At the start: 115 parts, among them J1 Barrel_Jack, J2 MIDI OUT, J3 MIDI IN, J4 AudioJack2, J5 AudioJack2, J6 AudioJack2, J7 AudioJack2, J8 AudioJack2, J9 AudioJack2, P1 PTV09A-4020S-B103, P10 PTV09A-4020S-B103, P11 PTV09A-4020S-B103, P12 PTV09A-4020S-B103, P13 PTV09A-4020S-B103, P14 PTV09A-4020S-B103, P15 PTV09A-4020S-B103, P16 PTV09A-4020S-B103, P17 PTV09A-4020S-B103, P18 PTV09A-4020S-B103, P19 PTV09A-4020S-B103, P2 PTV09A-4020S-B103, P20 PTV09A-4020S-B103, P21 PTV09A-4020S-B103, P22 PTV09A-4020S-B103, P23 PTV09A-4020S-B103, P24 PTV09A-4020S-B103, P25 PTV09A-4020S-B103, P26 PTV09A-4020S-B103, P27 PTV09A-4020S-B103, P28 PTV09A-4020S-B103, P29 PTV09A-4020S-B103, P3 PTV09A-4020S-B103, P30 PTV09A-4020S-B103, P31 PTV09A-4020S-B103, P32 PTV09A-4020S-B103, P33 PTV09A-4020S-B103, P34 PTV09A-4020S-B103, P35 PTV09A-4020S-B103, P36 PTV09A-4020S-B103, P37 PTV09A-4020S-B103, P38 PTV09A-4020S-B103, P39 PTV09A-4020S-B103, P4 PTV09A-4020S-B103, P40 PTV09A-4020S-B103, P41 PTV09A-4020S-B103, P42 PTV09A-4020S-B103, P5 PTV09A-4020S-B103, P6 PTV09A-4020S-B103, P7 PTV09A-4020S-B103, P8 PTV09A-4020S-B103, P9 PTV09A-4020S-B103, SW1 SW_MEC_5E, SW2 SW_MEC_5E, SW3 SW_MEC_5E, SW4 SW_MEC_5E, SW5 SW_MEC_5E, SW6 SW_MEC_5E, U1 teensy 4.0, U10 6N138, U2 TXB0108DQSR, U3 74HC4051, U4 74HC4051, U5 74HC4051, U6 74HC4051, U7 74HC4051, U8 74HC4051, U9 74HC4051

Commit message: board
circuit diagram
Parts:
- removed P1, P10, P11, P12, P13, P14, P15, P16, P17, P18, P19, P2, P20, P21, P22, P23, P24, P25, P26, P27, P28, P29, P3, P30, P31, P32, P33, P34, P35, P36, P37, P38, P39, P4, P40, P41, P42, P5, P6, P7, P8, P9: PTV09A-4020S-B103, TO_B103, symbol 10K Potentiometer_digikey:PTV09A-4020S-B103
- added R10, R11, R12, R13, R14, R15, R16, R17, R18, R19, R20, R21, R22, R23, R24, R25, R26, R27, R28, R29, R30, R31, R32, R33, R34, R35, R36, R37, R38, R39, R40, R41, R42, R43, R44, R45, R46, R5, R6, R7, R8, R9: R_Variable, symbol Device:R_Variable
Connections:
- net 5VDC: now also SW1.2, R10.2, R11.2, R12.2, R13.2, R14.2, R15.2, R16.2, R17.2, R18.2, R19.2, R20.2, R21.2, R22.2, R23.2, R24.2, R25.2, R26.2, R27.2, R28.2, R29.2, R30.2, R31.2, R32.2, R33.2, R34.2, R35.2, R36.2, R37.2, R38.2, R39.2, R40.2, R41.2, R42.2, R43.2, R44.2, R45.2, R46.2, R5.2, R6.2, R7.2, R8.2, R9.2; no longer SW1.1
- net B1_1: now also R8.1
- net B1_2: now also R13.1
- net B1_3: now also R17.1
- net B1_4: now also R21.1
- net B1_5: now also R25.1
- net B1_6: now also R30.1
- net B1_7: now also R33.1
- net B2_1: now also R35.1
- net B2_2: now also R39.1
- net B2_3: now also R43.1
- net B2_4: now also R5.1
- net B2_5: now also R11.1
- net B2_6: now also R15.1
- net B2_7: now also R19.1
- net B3_1: now also R23.1
- net B3_2: now also R27.1
- net B3_3: now also R31.1
- net B3_4: now also R36.1
- net B3_5: now also R40.1
- net B3_6: now also R44.1
- net B3_7: now also R6.1
- net B4_1: now also R12.1
- net B4_2: now also R16.1
- net B4_3: now also R20.1
- net B4_4: now also R24.1
- net B4_5: now also R28.1
- net B4_6: now also R32.1
- net B4_7: now also R37.1
- net B5_1: now also R41.1
- net B5_2: now also R45.1
- net B5_3: now also R7.1
- net B5_4: now also R14.1
- net B5_5: now also R18.1
- net B5_6: now also R22.1
- net B5_7: now also R26.1
- net B6_1: now also R29.1
- net B6_2: now also R34.1
- net B6_3: now also R38.1
- net B6_4: now also R42.1
- net B6_5: now also R46.1
- net B6_6: now also R9.1
- net B6_7: now also R10.1
Other:
- moved on the sheet: SW1, SW2, SW3, SW4, SW5, SW6

Commit message: moar
booooooard
Parts:
- removed J4, J5, J6, J7, J8, J9: AudioJack2, symbol Connector:AudioJack2
- removed R10, R11, R12, R13, R14, R15, R16, R17, R18, R19, R20, R21, R22, R23, R24, R25, R26, R27, R28, R29, R30, R31, R32, R33, R34, R35, R36, R37, R38, R39, R40, R41, R42, R43, R44, R45, R46, R5, R6, R7, R8, R9: R_Variable, symbol Device:R_Variable
- removed SW1, SW2, SW3, SW4, SW5, SW6: SW_MEC_5E, symbol Switch:SW_MEC_5E
- added J4, J5, J6, J7, J8, J9: MJ-3502, audioJack:CONN_MJ-3502, symbol audioJack-DIGIKEY:MJ-3502
- added R10, R11, R12, R13, R14, R15, R16, R17, R18, R19, R20, R21, R22, R23, R24, R25, R26, R27, R28, R29, R30, R31, R32, R33, R34, R35, R36, R37, R38, R39, R40, R41, R42, R43, R44, R45, R46, R5, R6, R7, R8, R9: R_Potentiometer, Potentiometer_THT:Potentiometer_Alps_RK09K_Single_Vertical, symbol Device:R_Potentiometer
- added S1, S2, S3, S4, S5, S6: B3F-4055, Button_Switch_THT:SW_TH_Tactile_Omron_B3F-10xx, symbol longButton:B3F-4055
- D1, D10, D11, D12, D13, D14, D15, D16, D17, D18, D19, D2, D20, D21, D22, D23, D24, D25, D26, D27, D28, D29, D3, D30, D31, D32, D33, D34, D35, D36, D37, D38, D39, D4, D40, D41, D42, D5, D6, D7, D8, D9: footprint (none) -> LED_SMD:LED_SK6812MINI_PLCC4_3.5x3.5mm_P1.75mm
- J1: footprint (none) -> Connector_BarrelJack:BarrelJack_CUI_PJ-102AH_Horizontal
- J2, J3: footprint (none) -> midiJack:KYCON_KCDX-5S-N
- OLED1: footprint Qwiic_OLED_1.3in:OLED-1.3-128X64 -> Display:Adafruit_SSD1306
- R1, R2, R3, R4: footprint (none) -> Resistor_THT:R_Axial_DIN0204_L3.6mm_D1.6mm_P2.54mm_Vertical
- U1: footprint DEV-15583:MODULE_DEV-15583 -> teensy 4.0:MODULE_DEV-15583
- U10: footprint (none) -> Package_DIP:DIP-8_W7.62mm_Socket
- U3, U4, U5, U6, U7, U8, U9: footprint (none) -> cd74hc4051:N16
Connections:
- net GROUND is gone; now on net GND: D1.2 (GND), D10.2 (GND), D11.2 (GND), D12.2 (GND), D13.2 (GND), D14.2 (GND), D15.2 (GND), D16.2 (GND), D17.2 (GND), D18.2 (GND), D19.2 (GND), D2.2 (GND), D20.2 (GND), D21.2 (GND), D22.2 (GND), D23.2 (GND), D24.2 (GND), D25.2 (GND), D26.2 (GND), D27.2 (GND), D28.2 (GND), D29.2 (GND), D3.2 (GND), D30.2 (GND), D31.2 (GND), D32.2 (GND), D33.2 (GND), D34.2 (GND), D35.2 (GND), D36.2 (GND), D37.2 (GND), D38.2 (GND), D39.2 (GND), D4.2 (GND), D40.2 (GND), D41.2 (GND), D42.2 (GND), D5.2 (GND), D6.2 (GND), D7.2 (GND), D8.2 (GND), D9.2 (GND), J1.2, J2.2, OLED1.1 (GND@1), U1.G1, U1.G2, U10.5 (GND), U2.15 (GND), U3.6 (~{E}), U3.8 (GND), U4.6 (~{E}), U4.8 (GND), U5.6 (~{E}), U5.8 (GND), U6.6 (~{E}), U6.8 (GND), U7.6 (~{E}), U7.8 (GND), U8.6 (~{E}), U8.8 (GND), U9.6 (~{E}), U9.8 (GND)
- net Mux3B is gone; now on net MuxB3: U4.9 (S2)
- net A0: now also J7.3
- net A1: now also J6.3
- net A2: now also J5.3
- net A3: now also J4.3
- net A4: now also J8.3
- net A5: now also J9.3
- net B1_1: now also R5.2
- net B1_2: now also R6.2
- net B1_3: now also R7.2
- net B1_4: now also R8.2
- net B1_5: now also R9.2
- net B1_6: now also R10.2
- net B1_7: now also R11.2
- net B1_8: now also S1.3, S1.4
- net B2_1: now also R12.2
- net B2_2: now also R13.2
- net B2_3: now also R14.2
- net B2_4: now also R15.2
- net B2_5: now also R16.2
- net B2_6: now also R17.2
- net B2_7: now also R18.2
- net B2_8: now also S2.3, S2.4
- net B3_1: now also R19.2
- net B3_2: now also R20.2
- net B3_3: now also R21.2
- net B3_4: now also R22.2
- net B3_5: now also R23.2
- net B3_6: now also R24.2
- net B3_7: now also R25.2
- net B3_8: now also S3.3, S3.4
- net B4_1: now also R26.2
- net B4_2: now also R27.2
- net B4_3: now also R28.2
- net B4_4: now also R29.2
- net B4_5: now also R30.2
- net B4_6: now also R31.2
- net B4_7: now also R32.2
- net B4_8: now also S4.3, S4.4
- net B5_1: now also R33.2
- net B5_2: now also R34.2
- net B5_3: now also R35.2
- net B5_4: now also R36.2
- net B5_5: now also R37.2
- net B5_6: now also R38.2
- net B5_7: now also R39.2
- net B5_8: now also S5.3, S5.4
- net B6_1: now also R40.2
- net B6_2: now also R41.2
- net B6_3: now also R42.2
- net B6_4: now also R43.2
- net B6_5: now also R44.2
- net B6_6: now also R45.2
- net B6_7: now also R46.2
- net B6_8: now also S6.3, S6.4
- net GND: now also J4.1, J4.2, J5.1, J5.2, J6.1, J6.2, J7.1, J7.2, J8.1, J8.2, J9.1, J9.2, R10.3, R11.3, R12.3, R13.3, R14.3, R15.3, R16.3, R17.3, R18.3, R19.3, R20.3, R21.3, R22.3, R23.3, R24.3, R25.3, R26.3, R27.3, R28.3, R29.3, R30.3, R31.3, R32.3, R33.3, R34.3, R35.3, R36.3, R37.3, R38.3, R39.3, R40.3, R41.3, R42.3, R43.3, R44.3, R45.3, R46.3, R5.3, R6.3, R7.3, R8.3, R9.3; no longer U1.G3
- net LED_CNTRL: now also U2.11 (B8)
- net MuxB1: now also U2.14 (B5)
- net MuxB2: now also U2.13 (B6)
- net MuxB3: now also U2.12 (B7)
- net 5VDC renamed +5V
- net +5V: now also R10.1, R11.1, R12.1, R13.1, R14.1, R15.1, R16.1, R17.1, R18.1, R19.1, R20.1, R21.1, R22.1, R23.1, R24.1, R25.1, R26.1, R27.1, R28.1, R29.1, R30.1, R31.1, R32.1, R33.1, R34.1, R35.1, R36.1, R37.1, R38.1, R39.1, R40.1, R41.1, R42.1, R43.1, R44.1, R45.1, R46.1, R5.1, R6.1, R7.1, R8.1, R9.1, S1.1, S1.2, S2.1, S2.2, S3.1, S3.2, S4.1, S4.2, S5.1, S5.2, S6.1, S6.2
- no-connect marks 0 -> 25
Other:
- moved on the sheet: OLED1

Commit message: board
moar
Parts:
- removed OLED1: OLED1.3, Display:Adafruit_SSD1306, symbol Qwiic_OLED_1.3in-eagle-import:OLED1.3
- removed S1, S2, S3, S4, S5, S6: B3F-4055, Button_Switch_THT:SW_TH_Tactile_Omron_B3F-10xx, symbol longButton:B3F-4055
- added J10: I2C_STANDARDJS-1MM, Connector_JST:JST_EH_S4B-EH_1x04_P2.50mm_Horizontal, symbol Qwiic_OLED_1.3in-eagle-import:I2C_STANDARDJS-1MM
- added SW1, SW2, SW3, SW4, SW5, SW6: SW_MEC_5E, Button_Switch_THT:SW_TH_Tactile_Omron_B3F-10xx, symbol Switch:SW_MEC_5E
Connections:
- net +5V: now also J10.2 (VCC), SW1.1, SW2.1, SW3.1, SW4.1, SW5.1, SW6.1
- net B1_8: now also SW1.4 (A)
- net B2_8: now also SW2.4 (A)
- net B3_8: now also SW3.4 (A)
- net B4_8: now also SW4.4 (A)
- net B5_8: now also SW5.4 (A)
- net B6_8: now also SW6.4 (A)
- net GND: now also U1.G3, J10.1 (GND)
- net SCL: now also J10.4 (SCL)
- net SDA: now also J10.3 (SDA)
- no-connect marks 25 -> 38

Commit message: circuit/board
finalizing power regulation
Parts:
- added C1, C2: CAP_CERAMIC0402, Capacitor_THT:C_Disc_D4.3mm_W1.9mm_P5.00mm, symbol BenzKnobz-eagle-import:CAP_CERAMIC0402
- added D44: 1N4007, Diode_THT:D_DO-41_SOD81_P10.16mm_Horizontal, symbol Diode:1N4007
- added SW7: SW_Push_SPDT, Button_Switch_THT:SW_PUSH_6mm, symbol Switch:SW_Push_SPDT
- added TH1: Thermistor, Capacitor_THT:C_Disc_D9.0mm_W5.0mm_P7.50mm, symbol Device:Thermistor
- added U11: LM317_TO-220, Package_TO_SOT_THT:TO-220-3_Vertical, symbol Regulator_Linear:LM317_TO-220
Connections:
- net +5V: no longer D1.3 (VDD), D10.3 (VDD), D11.3 (VDD), D12.3 (VDD), D13.3 (VDD), D14.3 (VDD), D15.3 (VDD), D16.3 (VDD), D17.3 (VDD), D18.3 (VDD), D19.3 (VDD), D2.3 (VDD), D20.3 (VDD), D21.3 (VDD), D22.3 (VDD), D23.3 (VDD), D24.3 (VDD), D25.3 (VDD), D26.3 (VDD), D27.3 (VDD), D28.3 (VDD), D29.3 (VDD), D3.3 (VDD), D30.3 (VDD), D31.3 (VDD), D32.3 (VDD), D33.3 (VDD), D34.3 (VDD), D35.3 (VDD), D36.3 (VDD), D37.3 (VDD), D38.3 (VDD), D39.3 (VDD), D4.3 (VDD), D40.3 (VDD), D41.3 (VDD), D42.3 (VDD), D5.3 (VDD), D6.3 (VDD), D7.3 (VDD), D8.3 (VDD), D9.3 (VDD), J10.2 (VCC), R10.1, R11.1, R12.1, R13.1, R14.1, R15.1, R16.1, R17.1, R18.1, R19.1, R2.1, R20.1, R21.1, R22.1, R23.1, R24.1, R25.1, R26.1, R27.1, R28.1, R29.1, R30.1, R31.1, R32.1, R33.1, R34.1, R35.1, R36.1, R37.1, R38.1, R39.1, R4.1, R40.1, R41.1, R42.1, R43.1, R44.1, R45.1, R46.1, R5.1, R6.1, R7.1, R8.1, R9.1, SW1.1, SW2.1, SW3.1, SW4.1, SW5.1, SW6.1, U1.VIN, U10.8 (VCC), U2.16 (VCCB), U3.16 (VCC), U4.16 (VCC), U5.16 (VCC), U6.16 (VCC), U7.16 (VCC), U8.16 (VCC), U9.16 (VCC)
- net GND: now also C1.2 (P$2), C2.2 (P$2), SW7.3 (C)
- new net: U1.VIN, U11.2 (VO), U2.16 (VCCB)
- new net: C1.1 (P$1), C2.1 (P$1), D44.1 (K), U11.3 (VI)
- new net: D44.2 (A), SW7.1 (A)
- new net: SW7.2 (B), TH1.2
- new net 5VDC: D1.3 (VDD), D10.3 (VDD), D11.3 (VDD), D12.3 (VDD), D13.3 (VDD), D14.3 (VDD), D15.3 (VDD), D16.3 (VDD), D17.3 (VDD), D18.3 (VDD), D19.3 (VDD), D2.3 (VDD), D20.3 (VDD), D21.3 (VDD), D22.3 (VDD), D23.3 (VDD), D24.3 (VDD), D25.3 (VDD), D26.3 (VDD), D27.3 (VDD), D28.3 (VDD), D29.3 (VDD), D3.3 (VDD), D30.3 (VDD), D31.3 (VDD), D32.3 (VDD), D33.3 (VDD), D34.3 (VDD), D35.3 (VDD), D36.3 (VDD), D37.3 (VDD), D38.3 (VDD), D39.3 (VDD), D4.3 (VDD), D40.3 (VDD), D41.3 (VDD), D42.3 (VDD), D5.3 (VDD), D6.3 (VDD), D7.3 (VDD), D8.3 (VDD), D9.3 (VDD), J10.2 (VCC), R10.1, R11.1, R12.1, R13.1, R14.1, R15.1, R16.1, R17.1, R18.1, R19.1, R2.1, R20.1, R21.1, R22.1, R23.1, R24.1, R25.1, R26.1, R27.1, R28.1, R29.1, R30.1, R31.1, R32.1, R33.1, R34.1, R35.1, R36.1, R37.1, R38.1, R39.1, R4.1, R40.1, R41.1, R42.1, R43.1, R44.1, R45.1, R46.1, R5.1, R6.1, R7.1, R8.1, R9.1, SW1.1, SW2.1, SW3.1, SW4.1, SW5.1, SW6.1, U10.8 (VCC), U3.16 (VCC), U4.16 (VCC), U5.16 (VCC), U6.16 (VCC), U7.16 (VCC), U8.16 (VCC), U9.16 (VCC)
Other:
- moved on the sheet: J1

Commit message: kicad again
might need to restart layout
Connections:
- net 5VDC: now also SW1.2, SW2.2, SW3.2, SW4.2, SW5.2, SW6.2, TH1.1
- net B1_8: now also SW1.3 (K)
- net B2_8: now also SW2.3 (K)
- net B3_8: now also SW3.3 (K)
- net B4_8: now also SW4.3 (K)
- net B5_8: now also SW5.3 (K)
- net B6_8: now also SW6.3 (K)
- net MuxBD1: now reaches U3.13 (A0), U4.3 (A)
- net MuxBD5: now reaches U3.1 (A4), U9.3 (A)
- net MuxA3: now reaches U2.17 (B4), U3.9 (S2)
- net MuxA2: now reaches U2.18 (B3), U3.10 (S1)
- net MuxA1: now reaches U2.19 (B2), U3.11 (S0)
- net MUX_OUT: now reaches U2.20 (B1), U3.3 (A)
- net MuxBD2: now reaches U3.14 (A1), U5.3 (A)
- net MuxBD3: now reaches U3.15 (A2), U6.3 (A)
- net MuxBD6: now reaches U3.5 (A5), U8.3 (A)
- net MuxBD4: now reaches U3.12 (A3), U7.3 (A)
- no-connect marks 38 -> 25
Other:
- moved on the sheet: J10, J4, J5, J6, J7, J8, J9, U3

Commit message: two boards one git
two boards now - one for ui, the other for ics and io
Parts:
- removed D1, D10, D11, D12, D13, D14, D15, D16, D17, D18, D19, D2, D20, D21, D22, D23, D24, D25, D26, D27, D28, D29, D3, D30, D31, D32, D33, D34, D35, D36, D37, D38, D39, D4, D40, D41, D42, D5, D6, D7, D8, D9: NeoPixel_THT, LED_SMD:LED_SK6812MINI_PLCC4_3.5x3.5mm_P1.75mm, symbol LED:NeoPixel_THT
- removed R10, R11, R12, R13, R14, R15, R16, R17, R18, R19, R20, R21, R22, R23, R24, R25, R26, R27, R28, R29, R30, R31, R32, R33, R34, R35, R36, R37, R38, R39, R40, R41, R42, R43, R44, R45, R46, R5, R6, R7, R8, R9: R_Potentiometer, Potentiometer_THT:Potentiometer_Alps_RK09K_Single_Vertical, symbol Device:R_Potentiometer
- removed SW1, SW2, SW3, SW4, SW5, SW6: SW_MEC_5E, Button_Switch_THT:SW_TH_Tactile_Omron_B3F-10xx, symbol Switch:SW_MEC_5E
- removed U2: TXB0108DQSR, Package_SON:USON-20_2x4mm_P0.4mm, symbol Logic_LevelTranslator:TXB0108DQSR
- added J11: Conn_01x02, Connector_PinHeader_1.00mm:PinHeader_1x02_P1.00mm_Vertical, symbol Connector_Generic:Conn_01x02
- added J12, J13, J14, J15, J16, J17, J18: Conn_01x07, Connector_PinHeader_1.00mm:PinHeader_1x07_P1.00mm_Vertical, symbol Connector_Generic:Conn_01x07
- added U12, U2: CD74HC4050E, cd74hc4051:N16, symbol cd74hc4050e:CD74HC4050E
Connections:
- net 5VDC: now also J11.1 (Pin_1), U2.1 (VCC)
- net GND: now also J11.2 (Pin_2), U12.8 (GND), U2.8 (GND)
- net M1: now also U2.3 (1A)
- net M2: now also U2.5 (2A)
- net M3: now also U2.7 (3A)
- net M4: now also U2.9 (4A)
- net M5: now also U2.11 (5A)
- net M6: now also U2.14 (6A)
- net MUX_OUT: now also U12.3 (1A)
- net MUX_READ: now also U12.2 (1Y)
- net MuxA1: now also U2.2 (1Y)
- net MuxA2: now also U2.4 (2Y)
- net MuxA3: now also U2.6 (3Y)
- net MuxB1: now also U2.10 (4Y)
- net MuxB2: now also U2.12 (5Y)
- net MuxB3: now also U2.15 (6Y)
- net 3VDC: now reaches U1.3.3V_2
- net 3VDC: now also U12.1 (VCC)
- no-connect marks 25 -> 39
Other:
- removed sheet UI Sheet1
- removed sheet UI Sheet2
- moved on the sheet: J4, J8

Commit message: brd
moar - almost completely laid out
Parts:
- removed J10: I2C_STANDARDJS-1MM, Connector_JST:JST_EH_S4B-EH_1x04_P2.50mm_Horizontal, symbol Qwiic_OLED_1.3in-eagle-import:I2C_STANDARDJS-1MM
- removed J11: Conn_01x02, Connector_PinHeader_1.00mm:PinHeader_1x02_P1.00mm_Vertical, symbol Connector_Generic:Conn_01x02
- removed J12, J13, J14, J15, J16, J17, J18: Conn_01x07, Connector_PinHeader_1.00mm:PinHeader_1x07_P1.00mm_Vertical, symbol Connector_Generic:Conn_01x07
- added J10, J11: Conn_01x03, Connector_PinHeader_1.00mm:PinHeader_1x03_P1.00mm_Vertical, symbol Connector_Generic:Conn_01x03
- added J12, J13, J14, J15, J16, J17: Conn_02x04_Odd_Even_Shielded, Connector_PinHeader_1.00mm:PinHeader_2x04_P1.00mm_Vertical, symbol Connector_Generic:Conn_02x04_Odd_Even
Connections:
- net 3VDC: now also J11.1 (Pin_1)
- net 5VDC: now also J11.3 (Pin_3)
- net B1_1: now also J12.1 (Pin_1)
- net B1_2: now also J12.2 (Pin_2)
- net B1_3: now also J12.3 (Pin_3)
- net B1_4: now also J12.4 (Pin_4)
- net B1_5: now also J12.5 (Pin_5)
- net B1_6: now also J12.6 (Pin_6)
- net B1_7: now also J12.7 (Pin_7)
- net B1_8: now also J12.8 (Pin_8)
- net B2_1: now also J13.1 (Pin_1)
- net B2_2: now also J13.2 (Pin_2)
- net B2_3: now also J13.3 (Pin_3)
- net B2_4: now also J13.4 (Pin_4)
- net B2_5: now also J13.5 (Pin_5)
- net B2_6: now also J13.6 (Pin_6)
- net B2_7: now also J13.7 (Pin_7)
- net B2_8: now also J13.8 (Pin_8)
- net B3_1: now also J14.1 (Pin_1)
- net B3_2: now also J14.2 (Pin_2)
- net B3_3: now also J14.3 (Pin_3)
- net B3_4: now also J14.4 (Pin_4)
- net B3_5: now also J14.5 (Pin_5)
- net B3_6: now also J14.6 (Pin_6)
- net B3_7: now also J14.7 (Pin_7)
- net B3_8: now also J14.8 (Pin_8)
- net B4_1: now also J15.1 (Pin_1)
- net B4_2: now also J15.2 (Pin_2)
- net B4_3: now also J15.3 (Pin_3)
- net B4_4: now also J15.4 (Pin_4)
- net B4_5: now also J15.5 (Pin_5)
- net B4_6: now also J15.6 (Pin_6)
- net B4_7: now also J15.7 (Pin_7)
- net B4_8: now also J15.8 (Pin_8)
- net B5_1: now also J16.1 (Pin_1)
- net B5_2: now also J16.2 (Pin_2)
- net B5_3: now also J16.3 (Pin_3)
- net B5_4: now also J16.4 (Pin_4)
- net B5_5: now also J16.5 (Pin_5)
- net B5_6: now also J16.6 (Pin_6)
- net B5_7: now also J16.7 (Pin_7)
- net B5_8: now also J16.8 (Pin_8)
- net B6_1: now also J17.1 (Pin_1)
- net B6_2: now also J17.2 (Pin_2)
- net B6_3: now also J17.3 (Pin_3)
- net B6_4: now also J17.4 (Pin_4)
- net B6_5: now also J17.5 (Pin_5)
- net B6_6: now also J17.6 (Pin_6)
- net B6_7: now also J17.7 (Pin_7)
- net B6_8: now also J17.8 (Pin_8)
- net GND: now also J11.2 (Pin_2)
- net LED: now also J10.3 (Pin_3)
- net MUX_OUT: no longer U12.3 (1A)
- net MUX_READ: now also U12.10 (4Y), U12.12 (5Y), U12.15 (6Y), U12.4 (2Y), U12.6 (3Y)
- net MuxBD1: now also U12.3 (1A)
- net MuxBD2: now also U12.5 (2A)
- net MuxBD3: now also U12.7 (3A)
- net MuxBD4: now also U12.9 (4A)
- net MuxBD5: now also U12.11 (5A), U8.3 (A); no longer U9.3 (A)
- net MuxBD6: now also U12.14 (6A), U9.3 (A); no longer U8.3 (A)
- net SCL: now also J10.1 (Pin_1)
- net SDA: now also J10.2 (Pin_2)
- no-connect marks 39 -> 27
Other:
- moved on the sheet: J2, J4, J5, J6, J7, J8, J9, R3, R4, U4, U5
