File: hardware/BTN_42/btnBRD/btnBRD.kicad_sch (KiCad schematic)
At the start: 110 parts, among them J1 Jack-DC, J10 Display Jumper, J2 DIN-5, J3 DIN-5, J4 AudioJack2, J5 AudioJack2, J6 AudioJack2, J7 AudioJack2, J8 AudioJack2, J9 AudioJack2, SW1 SW_Push, SW10 SW_Push, SW11 SW_Push, SW12 SW_Push, SW13 SW_Push, SW14 SW_Push, SW15 SW_Push, SW16 SW_Push, SW17 SW_Push, SW18 SW_Push, SW19 SW_Push, SW2 SW_Push, SW20 SW_Push, SW21 SW_Push, SW22 SW_Push, SW23 SW_Push, SW24 SW_Push, SW25 SW_Push, SW26 SW_Push, SW27 SW_Push, SW28 SW_Push, SW29 SW_Push, SW3 SW_Push, SW30 SW_Push, SW31 SW_Push, SW32 SW_Push, SW33 SW_Push, SW34 SW_Push, SW35 SW_Push, SW36 SW_Push, SW37 SW_Push, SW38 SW_Push, SW39 SW_Push, SW4 SW_Push, SW40 SW_Push, SW41 SW_Push, SW42 SW_Push, SW43 SW_Push, SW44 SW_Push, SW45 SW_Push, SW46 SW_Push, SW47 SW_Push, SW48 SW_Push, SW5 SW_Push, SW6 SW_Push, SW7 SW_Push, SW8 SW_Push, SW9 SW_Push, U1 brain, U2 CD74HC4067M, U3 CD74HC4067M

Commit message: brdMIdi
Parts:
- removed R5, R6: 10k, Resistor_THT:R_Axial_DIN0204_L3.6mm_D1.6mm_P2.54mm_Vertical, symbol Device:R
- added C2: 10uF, Capacitor_THT:CP_Radial_D4.0mm_P2.00mm, symbol Device:C
- added C? (x2): 100nF, Capacitor_THT:CP_Radial_D4.0mm_P2.00mm, symbol Device:C
- added D43: 1N4148, Diode_THT:D_DO-35_SOD27_P7.62mm_Horizontal, symbol Diode:1N4148
- added RV? (x2): R_Potentiometer, symbol Device:R_Potentiometer
- added U4: TXB0108DQSR, Package_SON:USON-20_2x4mm_P0.4mm, symbol Logic_LevelTranslator:TXB0108DQSR
- added U5: 6N138, symbol Isolator:6N138
- J2: value DIN-5 -> MIDI-IN
- J3: value DIN-5 -> MIDI-OUT
- R1, R3, R4: value 10k -> 220; footprint Resistor_THT:R_Axial_DIN0204_L3.6mm_D1.6mm_P2.54mm_Vertical -> (none)
- R2: value 10k -> 4.7k; footprint Resistor_THT:R_Axial_DIN0204_L3.6mm_D1.6mm_P2.54mm_Vertical -> (none)
Connections:
- net +5V: now also R1.2, R4.1, C2.2, U4.16 (VCCB), U5.8 (VCC); no longer U2.24 (VCC), U3.24 (VCC)
- net 3VDC: now also SW43.2, SW43.4, SW44.2, SW44.4, SW45.2, SW45.4, SW46.2, SW46.4, SW47.2, SW47.4, SW48.2, SW48.4, U1.3.3V_2, U2.24 (VCC), U3.24 (VCC), RV?.1, RV?.1, U4.5 (VCCA); no longer R1.2, R2.2, R3.2, R4.2
- net Ctrl1: now also U2.22 (I9); no longer R1.1, U1.0
- net Ctrl2: now also U2.23 (I8); no longer R2.1, U1.1
- net Ctrl3: now also U2.2 (I7); no longer R3.1, U1.2
- net Ctrl4: now also U3.23 (I8); no longer R4.1, U1.3
- net Ctrl5: now also U3.2 (I7); no longer U1.4
- net Ctrl6: now also U3.3 (I6); no longer U1.5
- net GND: now also J2.2, J3.2, R2.1, C2.1, C?.1, C?.1, RV?.3, RV?.3, U4.15 (GND), U5.5 (GND); no longer SW43.2, SW43.4, SW44.2, SW44.4, SW45.2, SW45.4, SW46.2, SW46.4, SW47.2, SW47.4, SW48.2, SW48.4, U2.1 (COM), U3.1 (COM)
- net LED: now also U4.1 (A1); no longer D1.4 (DIN)
- net MuxC1: now also U1.8, U3.10 (S0); no longer U1.10, U3.11 (S1)
- net MuxC2: now also U1.9, U3.11 (S1); no longer U1.11, U3.14 (S2)
- net MuxC3: now also U1.10, U3.14 (S2); no longer U1.12, U3.13 (S3)
- net MuxR1: now also U1.2, U2.10 (S0); no longer U1.7, U2.11 (S1)
- net MuxR2: now also U1.3, U2.11 (S1); no longer U1.8, U2.14 (S2)
- net MuxR3: now also U1.4, U2.14 (S2); no longer U1.9, U2.13 (S3)
- net MIDI_OUT: now reaches J3.4
- net MIDI_OUT: now also U4.18 (B3)
- net at J3.5: now also R4.2
- net fp2: now reaches U3.22 (I9)
- net fp2: now also RV?.2
- net fp1: now reaches U2.21 (I10)
- net fp1: now also RV?.2
- net at J2.4: now also R3.2
- net at J2.5: now also D43.2 (A), U5.3 (C2)
- net MuxREADcol renamed MRC
- net MRC: now also U3.1 (COM), C?.2; no longer U3.10 (S0)
- net MuxREADrow renamed MRR
- net MRR: now also U2.1 (COM), C?.2; no longer U2.10 (S0)
- new net: R2.2, U5.7 (VO1)
- new net: D43.1 (K), R3.1, U5.2 (C1)
- new net LEDcntrl: D1.4 (DIN), U4.20 (B1)
- new net MIDI_IN: R1.1, U4.19 (B2), U5.6 (VO2)
- new net MIDIi3: U1.0, U4.2 (A2)
- new net MIDIo3: U1.1, U4.3 (A3)
- new net MuxC4: U1.11, U3.13 (S3)
- new net MuxR4: U1.5, U2.13 (S3)
Other:
- moved on the sheet: J4, J5, J6, J7, J8, J9, U1, U2

Commit message: brddd
Parts:
- added RV3: 10k - main, Potentiometer_THT:Potentiometer_Alps_RK09L_Single_Vertical, symbol Device:R_Potentiometer
- C1: footprint Capacitor_THT:CP_Radial_D4.0mm_P2.00mm -> Capacitor_THT:C_Disc_D3.4mm_W2.1mm_P2.50mm
- C2: value 10uF -> 470uF; footprint Capacitor_THT:CP_Radial_D4.0mm_P2.00mm -> Capacitor_THT:C_Disc_D3.4mm_W2.1mm_P2.50mm
- C3, C4: renamed from C?; footprint Capacitor_THT:CP_Radial_D4.0mm_P2.00mm -> Capacitor_THT:C_Disc_D3.4mm_W2.1mm_P2.50mm
- R1, R2, R3, R4: footprint (none) -> Resistor_THT:R_Axial_DIN0204_L3.6mm_D1.6mm_P2.54mm_Vertical
- RV1: renamed from RV?; value R_Potentiometer -> 10k - ff; footprint (none) -> Potentiometer_THT:Potentiometer_Alps_RK09L_Single_Vertical
- RV2: renamed from RV?; value R_Potentiometer -> 10k - q; footprint (none) -> Potentiometer_THT:Potentiometer_Alps_RK09L_Single_Vertical
- SW1: value SW_Push -> 1x1; symbol Switch:SW_Push_Dual -> Switch:SW_Push
- SW10: value SW_Push -> 3x2; symbol Switch:SW_Push_Dual -> Switch:SW_Push
- SW11: value SW_Push -> 4x2; symbol Switch:SW_Push_Dual -> Switch:SW_Push
- SW12: value SW_Push -> 5x2; symbol Switch:SW_Push_Dual -> Switch:SW_Push
- SW13: value SW_Push -> 6x2; symbol Switch:SW_Push_Dual -> Switch:SW_Push
- SW14: value SW_Push -> 7x2; symbol Switch:SW_Push_Dual -> Switch:SW_Push
- SW15: value SW_Push -> 1x3; symbol Switch:SW_Push_Dual -> Switch:SW_Push
- SW16: value SW_Push -> 2x3; symbol Switch:SW_Push_Dual -> Switch:SW_Push
- SW17: value SW_Push -> 3x3; symbol Switch:SW_Push_Dual -> Switch:SW_Push
- SW18: value SW_Push -> 4x3; symbol Switch:SW_Push_Dual -> Switch:SW_Push
- SW19: value SW_Push -> 5x3; symbol Switch:SW_Push_Dual -> Switch:SW_Push
- SW2: value SW_Push -> 2x1; symbol Switch:SW_Push_Dual -> Switch:SW_Push
- SW20: value SW_Push -> 6x3; symbol Switch:SW_Push_Dual -> Switch:SW_Push
- SW21: value SW_Push -> 7x3; symbol Switch:SW_Push_Dual -> Switch:SW_Push
- SW22: value SW_Push -> 1x4; symbol Switch:SW_Push_Dual -> Switch:SW_Push
- SW23: value SW_Push -> 2x4; symbol Switch:SW_Push_Dual -> Switch:SW_Push
- SW24: value SW_Push -> 3x4; symbol Switch:SW_Push_Dual -> Switch:SW_Push
- SW25: value SW_Push -> 4x4; symbol Switch:SW_Push_Dual -> Switch:SW_Push
- SW26: value SW_Push -> 5x4; symbol Switch:SW_Push_Dual -> Switch:SW_Push
- SW27: value SW_Push -> 6x4; symbol Switch:SW_Push_Dual -> Switch:SW_Push
- SW28: value SW_Push -> 7x4; symbol Switch:SW_Push_Dual -> Switch:SW_Push
- SW29: value SW_Push -> 1x5; symbol Switch:SW_Push_Dual -> Switch:SW_Push
- SW3: value SW_Push -> 3x1; symbol Switch:SW_Push_Dual -> Switch:SW_Push
- SW30: value SW_Push -> 2x5; symbol Switch:SW_Push_Dual -> Switch:SW_Push
- SW31: value SW_Push -> 3x5; symbol Switch:SW_Push_Dual -> Switch:SW_Push
- SW32: value SW_Push -> 4x5; symbol Switch:SW_Push_Dual -> Switch:SW_Push
- SW33: value SW_Push -> 5x5; symbol Switch:SW_Push_Dual -> Switch:SW_Push
- SW34: value SW_Push -> 6x5; symbol Switch:SW_Push_Dual -> Switch:SW_Push
- SW35: value SW_Push -> 7x5; symbol Switch:SW_Push_Dual -> Switch:SW_Push
- SW36: value SW_Push -> 1x6; symbol Switch:SW_Push_Dual -> Switch:SW_Push
- SW37: value SW_Push -> 2x6; symbol Switch:SW_Push_Dual -> Switch:SW_Push
- SW38: value SW_Push -> 3x6; symbol Switch:SW_Push_Dual -> Switch:SW_Push
- SW39: value SW_Push -> 4x6; symbol Switch:SW_Push_Dual -> Switch:SW_Push
- SW4: value SW_Push -> 4x1; symbol Switch:SW_Push_Dual -> Switch:SW_Push
- SW40: value SW_Push -> 5x6; symbol Switch:SW_Push_Dual -> Switch:SW_Push
- SW41: value SW_Push -> 6x6; symbol Switch:SW_Push_Dual -> Switch:SW_Push
- SW42: value SW_Push -> 7x6; symbol Switch:SW_Push_Dual -> Switch:SW_Push
- SW43: value SW_Push -> cntrl1; symbol Switch:SW_Push_Dual -> Switch:SW_Push
- SW44: value SW_Push -> cntrl2; symbol Switch:SW_Push_Dual -> Switch:SW_Push
- SW45: value SW_Push -> cntrl3; symbol Switch:SW_Push_Dual -> Switch:SW_Push
- SW46: value SW_Push -> cntrl4; symbol Switch:SW_Push_Dual -> Switch:SW_Push
- SW47: value SW_Push -> cntrl5; symbol Switch:SW_Push_Dual -> Switch:SW_Push
- SW48: value SW_Push -> cntrl6; symbol Switch:SW_Push_Dual -> Switch:SW_Push
- SW5: value SW_Push -> 5x1; symbol Switch:SW_Push_Dual -> Switch:SW_Push
- SW6: value SW_Push -> 6x1; symbol Switch:SW_Push_Dual -> Switch:SW_Push
- SW7: value SW_Push -> 7x1; symbol Switch:SW_Push_Dual -> Switch:SW_Push
- SW8: value SW_Push -> 1x2; symbol Switch:SW_Push_Dual -> Switch:SW_Push
- SW9: value SW_Push -> 2x2; symbol Switch:SW_Push_Dual -> Switch:SW_Push
- U1: value brain -> brain - teensy 4.0
- U2: value CD74HC4067M -> digital mux - 74hc4067m
- U3: value CD74HC4067M -> analog mux - 74hc4067m
- U5: footprint (none) -> Package_DIP:DIP-8_W7.62mm
Connections:
- net 3VDC: now also C3.2, C4.2, RV3.1; no longer SW1.2, SW1.4, SW10.2, SW10.4, SW11.2, SW11.4, SW12.2, SW12.4, SW13.2, SW13.4, SW14.2, SW14.4, SW15.2, SW15.4, SW16.2, SW16.4, SW17.2, SW17.4, SW18.2, SW18.4, SW19.2, SW19.4, SW2.2, SW2.4, SW20.2, SW20.4, SW21.2, SW21.4, SW22.2, SW22.4, SW23.2, SW23.4, SW24.2, SW24.4, SW25.2, SW25.4, SW26.2, SW26.4, SW27.2, SW27.4, SW28.2, SW28.4, SW29.2, SW29.4, SW3.2, SW3.4, SW30.2, SW30.4, SW31.2, SW31.4, SW32.2, SW32.4, SW33.2, SW33.4, SW34.2, SW34.4, SW35.2, SW35.4, SW36.2, SW36.4, SW37.2, SW37.4, SW38.2, SW38.4, SW39.2, SW39.4, SW4.2, SW4.4, SW40.2, SW40.4, SW41.2, SW41.4, SW42.2, SW42.4, SW43.4, SW44.4, SW45.4, SW46.4, SW47.4, SW48.4, SW5.2, SW5.4, SW6.2, SW6.4, SW7.2, SW7.4, SW8.2, SW8.4, SW9.2, SW9.4
- net Ctrl1: now also U3.8 (I1); no longer SW43.3, U2.22 (I9)
- net Ctrl2: now also U3.7 (I2); no longer SW44.3, U2.23 (I8)
- net Ctrl3: now also U3.6 (I3); no longer SW45.3, U2.2 (I7)
- net Ctrl4: now also U3.5 (I4); no longer SW46.3, U3.23 (I8)
- net Ctrl5: now also U3.4 (I5); no longer SW47.3, U3.2 (I7)
- net Ctrl6: no longer SW48.3
- net GND: now also U4.6 (OE), RV3.3
- net MRC: no longer C4.2
- net MRR: no longer C3.2
- net col1: now also SW1.2, SW2.2, SW3.2, SW4.2, SW5.2, SW6.2, SW7.2, U2.2 (I7); no longer SW1.3, SW2.3, SW3.3, SW4.3, SW5.3, SW6.3, SW7.3, U3.9 (I0)
- net col2: now also SW10.2, SW11.2, SW12.2, SW13.2, SW14.2, SW8.2, SW9.2, U2.23 (I8); no longer SW10.3, SW11.3, SW12.3, SW13.3, SW14.3, SW8.3, SW9.3, U3.8 (I1)
- net col3: now also SW15.2, SW16.2, SW17.2, SW18.2, SW19.2, SW20.2, SW21.2, U2.22 (I9); no longer SW15.3, SW16.3, SW17.3, SW18.3, SW19.3, SW20.3, SW21.3, U3.7 (I2)
- net col4: now also SW22.2, SW23.2, SW24.2, SW25.2, SW26.2, SW27.2, SW28.2, U2.21 (I10); no longer SW22.3, SW23.3, SW24.3, SW25.3, SW26.3, SW27.3, SW28.3, U3.6 (I3)
- net col5: now also SW29.2, SW30.2, SW31.2, SW32.2, SW33.2, SW34.2, SW35.2, U2.20 (I11); no longer SW29.3, SW30.3, SW31.3, SW32.3, SW33.3, SW34.3, SW35.3, U3.5 (I4)
- net col6: now also SW36.2, SW37.2, SW38.2, SW39.2, SW40.2, SW41.2, SW42.2, U2.19 (I12); no longer SW36.3, SW37.3, SW38.3, SW39.3, SW40.3, SW41.3, SW42.3, U3.4 (I5)
- net fp1: now also U3.9 (I0); no longer U2.21 (I10)
- net fp2: now also U3.2 (I7); no longer U3.22 (I9)
- net +5V renamed 5VDC
- new net main: RV3.2, U3.23 (I8)
- no-connect marks 0 -> 31
Other:
- note added: "12/03/25"
- note added: "5b"
- note added: "MOARkNOBS v2"
- moved on the sheet: C2, C3, C4, J10, J4, J5, J6, J7, J8, J9, RV1, RV2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
