File: hardware/BTN_42/btnBRD/_autosave-btnBRD.kicad_sch (KiCad schematic)
At the start: 117 parts, among them J1 Jack-DC, J10 Display Jumper, J2 MIDI-IN, J3 MIDI-OUT, J4 AudioJack2, J5 AudioJack2, J6 AudioJack2, J7 AudioJack2, J8 AudioJack2, J9 AudioJack2, SW1 1x1, SW10 3x2, SW11 4x2, SW12 5x2, SW13 6x2, SW14 7x2, SW15 1x3, SW16 2x3, SW17 3x3, SW18 4x3, SW19 5x3, SW2 2x1, SW20 6x3, SW21 7x3, SW22 1x4, SW23 2x4, SW24 3x4, SW25 4x4, SW26 5x4, SW27 6x4, SW28 7x4, SW29 1x5, SW3 3x1, SW30 2x5, SW31 3x5, SW32 4x5, SW33 5x5, SW34 6x5, SW35 7x5, SW36 1x6, SW37 2x6, SW38 3x6, SW39 4x6, SW4 4x1, SW40 5x6, SW41 6x6, SW42 7x6, SW43 cntrl1, SW44 cntrl2, SW45 cntrl3, SW46 cntrl4, SW47 cntrl5, SW48 cntrl6, SW5 5x1, SW6 6x1, SW7 7x1, SW8 1x2, SW9 2x2, U1 brain - teensy 4.0, U2 digital mux - 74hc4067m, U3 analog mux - 74hc4067m, U4 TXB0108DQSR, U5 6N138

Commit message: moar brd
Parts:
- gave numbers to parts that had none: 1
Changed lines of the file:
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@@
   (symbol (lib_id "Device:C") (at 30.48 101.6 90) (unit 1)
     (in_bom yes) (on_board yes) (fields_autoplaced)
-    (property "Reference" "C?" (id 0) (at 30.48 93.98 90))
+    (property "Reference" "C2" (id 0) (at 30.48 93.98 90))
     (property "Value" "470uF" (id 1) (at 30.48 96.52 90))
     (property "Footprint" "Capacitor_THT:C_Disc_D3.4mm_W2.1mm_P2.50mm" (id 2) (at 34.29 100.6348 0)
@@
       (reference "C1") (unit 1) (value "10uF") (footprint "Capacitor_THT:C_Disc_D3.4mm_W2.1mm_P2.50mm")
     )
+    (path "/fa98713f-8408-4b37-bc10-cdde37b53bbc"
+      (reference "C2") (unit 1) (value "470uF") (footprint "Capacitor_THT:C_Disc_D3.4mm_W2.1mm_P2.50mm")
+    )
     (path "/30ce997d-d322-4c2d-989b-144200741d5f"
       (reference "C3") (unit 1) (value "100nF") (footprint "Capacitor_THT:C_Disc_D3.4mm_W2.1mm_P2.50mm")
@@
       (reference "C4") (unit 1) (value "100nF") (footprint "Capacitor_THT:C_Disc_D3.4mm_W2.1mm_P2.50mm")
     )
-    (path "/fa98713f-8408-4b37-bc10-cdde37b53bbc"
-      (reference "C?") (unit 1) (value "470uF") (footprint "Capacitor_THT:C_Disc_D3.4mm_W2.1mm_P2.50mm")
-    )
     (path "/be0efb9a-75c1-4f9d-b9f9-f9896a850c66"
