File: hardware/BTN_42/btnBRD/btnBRD.kicad_pcb (KiCad board)
At the start: 2 copper layers, 110 parts, among them J1 Jack-DC, J10 Display Jumper, J2 DIN-5, J3 DIN-5, J4 AudioJack2, J5 AudioJack2, J6 AudioJack2, J7 AudioJack2, J8 AudioJack2, J9 AudioJack2, SW1 SW_Push, SW10 SW_Push, SW11 SW_Push, SW12 SW_Push, SW13 SW_Push, SW14 SW_Push, SW15 SW_Push, SW16 SW_Push, SW17 SW_Push, SW18 SW_Push, SW19 SW_Push, SW2 SW_Push, SW20 SW_Push, SW21 SW_Push, SW22 SW_Push, SW23 SW_Push, SW24 SW_Push, SW25 SW_Push, SW26 SW_Push, SW27 SW_Push, SW28 SW_Push, SW29 SW_Push, SW3 SW_Push, SW30 SW_Push, SW31 SW_Push, SW32 SW_Push, SW33 SW_Push, SW34 SW_Push, SW35 SW_Push, SW36 SW_Push, SW37 SW_Push, SW38 SW_Push, SW39 SW_Push, SW4 SW_Push, SW40 SW_Push, SW41 SW_Push, SW42 SW_Push, SW43 SW_Push, SW44 SW_Push, SW45 SW_Push, SW46 SW_Push, SW47 SW_Push, SW48 SW_Push, SW5 SW_Push, SW6 SW_Push, SW7 SW_Push, SW8 SW_Push, SW9 SW_Push, U1 brain, U2 CD74HC4067M, U3 CD74HC4067M

Commit message: brdMIdi
Parts:
- added C2: 10uF, Capacitor_THT:CP_Radial_D4.0mm_P2.00mm, F.Cu at (71.1, 43.2)
- added D43: 1N4148, Diode_THT:D_DO-35_SOD27_P7.62mm_Horizontal, F.Cu at (70.9, 38.6)
- added U4: TXB0108DQSR, Package_SON:USON-20_2x4mm_P0.4mm, F.Cu at (50.8, 45.7)
- J2: value DIN-5 -> MIDI-IN
- J3: value DIN-5 -> MIDI-OUT
- moved SW46 44.3 mm to (78.7, 160.4), turned to 180 degrees
- moved SW43 36.4 mm to (61.0, 160.4), turned to 180 degrees
- moved D42 33.5 mm to (189.8, 155.1)
- moved D36 33.5 mm to (189.7, 137.8)
- moved D30 32.5 mm to (189.8, 120.4)
- moved D12 32.5 mm to (189.8, 68.6)
- moved D18 32.4 mm to (189.8, 85.8)
- moved D24 32.3 mm to (189.8, 103.1)
- moved SW48 30.9 mm to (78.7, 121.9), turned to 180 degrees
- moved SW47 26.8 mm to (78.7, 141.2), turned to 180 degrees
- moved D35 22.8 mm to (170.6, 137.8)
- moved D41 22.8 mm to (170.5, 155.0)
- moved D29 21.8 mm to (170.6, 120.4)
- moved D25 21.7 mm to (94.0, 120.4)
- moved D11 21.6 mm to (170.6, 68.6)
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Connections:
- net MuxREADcol renamed MRC
- net MuxREADrow renamed MRR
- C1 pad 2: +5V -> 5VDC
- D1 pad 4: LED -> LEDcntrl
- D37 pad 1: +5V -> 5VDC
- J1 pad 1: +5V -> 5VDC
- J10 pad 1: +5V -> 5VDC
- J2 pad 2: unconnected-(J2-Pad2) -> GND
- J2 pad 4: unconnected-(J2-Pad4) -> Net-(J2-Pad4)
- J2 pad 5: unconnected-(J2-Pad5) -> Net-(J2-Pad5)
- J3 pad 2: unconnected-(J3-Pad2) -> GND
- J3 pad 4: unconnected-(J3-Pad4) -> MIDI_OUT
- J3 pad 5: unconnected-(J3-Pad5) -> Net-(J3-Pad5)
- SW43 pad 2: GND -> 3VDC
- SW44 pad 2: GND -> 3VDC
- SW45 pad 2: GND -> 3VDC
- SW46 pad 2: GND -> 3VDC
- SW47 pad 2: GND -> 3VDC
- SW48 pad 2: GND -> 3VDC
- U1 pad 0: Ctrl1 -> MIDIi3
- U1 pad 1: Ctrl2 -> MIDIo3
- U1 pad 2: Ctrl3 -> unconnected-(U1-Pad2)
- U1 pad 3: Ctrl4 -> unconnected-(U1-Pad3)
- U1 pad 3.3V_2: unconnected-(U1-Pad3.3V_2) -> 3VDC
- U1 pad 4: Ctrl5 -> unconnected-(U1-Pad4)
- U1 pad 5: Ctrl6 -> unconnected-(U1-Pad5)
- U1 pad VIN: +5V -> 5VDC
- U2 pad 2: unconnected-(U2-Pad2) -> Ctrl3
- U2 pad 22: unconnected-(U2-Pad22) -> Ctrl1
- U2 pad 23: unconnected-(U2-Pad23) -> Ctrl2
- U2 pad 24: +5V -> 3VDC
- U3 pad 2: unconnected-(U3-Pad2) -> Ctrl5
- U3 pad 23: unconnected-(U3-Pad23) -> Ctrl4
- U3 pad 24: +5V -> 3VDC
- U3 pad 3: unconnected-(U3-Pad3) -> Ctrl6
Routing:
- net 5VDC: track 0.00 -> 28.5 mm
- net +5V: track 28.5 -> 0.00 mm

Commit message: brddd
Parts:
- removed R5, R6: 10k, Resistor_THT:R_Axial_DIN0204_L3.6mm_D1.6mm_P2.54mm_Vertical
- added C3: 100nF, Capacitor_THT:C_Disc_D3.4mm_W2.1mm_P2.50mm, F.Cu at (48.3, 55.9)
- added C4: 100nF, Capacitor_THT:C_Disc_D3.4mm_W2.1mm_P2.50mm, F.Cu at (48.3, 78.7)
- added RV1: 10k - ff, Potentiometer_THT:Potentiometer_Alps_RK09L_Single_Vertical, F.Cu at (78.8, 91.2)
- added RV2: 10k - q, Potentiometer_THT:Potentiometer_Alps_RK09L_Single_Vertical, F.Cu at (78.8, 76.4)
- added RV3: 10k - main, Potentiometer_THT:Potentiometer_Alps_RK09L_Single_Vertical, F.Cu at (78.8, 61.6)
- added U5: 6N138, Package_DIP:DIP-8_W7.62mm, F.Cu at (68.6, 50.8)
- C1: footprint Capacitor_THT:CP_Radial_D4.0mm_P2.00mm -> Capacitor_THT:C_Disc_D3.4mm_W2.1mm_P2.50mm
- C2: value 10uF -> 470uF; footprint Capacitor_THT:CP_Radial_D4.0mm_P2.00mm -> Capacitor_THT:C_Disc_D3.4mm_W2.1mm_P2.50mm
- R1, R3, R4: value 10k -> 220
- R2: value 10k -> 4.7k
- SW1: value SW_Push -> 1x1
- SW10: value SW_Push -> 3x2
- SW11: value SW_Push -> 4x2
- SW12: value SW_Push -> 5x2
- SW13: value SW_Push -> 6x2
- SW14: value SW_Push -> 7x2
- SW15: value SW_Push -> 1x3
- SW16: value SW_Push -> 2x3
- SW17: value SW_Push -> 3x3
- SW18: value SW_Push -> 4x3
- SW19: value SW_Push -> 5x3
- SW2: value SW_Push -> 2x1
- SW20: value SW_Push -> 6x3
- SW21: value SW_Push -> 7x3
- SW22: value SW_Push -> 1x4
- SW23: value SW_Push -> 2x4
- SW24: value SW_Push -> 3x4
- SW25: value SW_Push -> 4x4
- SW26: value SW_Push -> 5x4
- SW27: value SW_Push -> 6x4
- SW28: value SW_Push -> 7x4
- SW29: value SW_Push -> 1x5
- SW3: value SW_Push -> 3x1
- SW30: value SW_Push -> 2x5
- SW31: value SW_Push -> 3x5
- SW32: value SW_Push -> 4x5
- SW33: value SW_Push -> 5x5
- SW34: value SW_Push -> 6x5
- SW35: value SW_Push -> 7x5
- SW36: value SW_Push -> 1x6
- SW37: value SW_Push -> 2x6
- SW38: value SW_Push -> 3x6
- SW39: value SW_Push -> 4x6
- SW4: value SW_Push -> 4x1
- SW40: value SW_Push -> 5x6
- SW41: value SW_Push -> 6x6
- SW42: value SW_Push -> 7x6
- SW43: value SW_Push -> cntrl1
- SW44: value SW_Push -> cntrl2
- SW45: value SW_Push -> cntrl3
- SW46: value SW_Push -> cntrl4
- SW47: value SW_Push -> cntrl5
- SW48: value SW_Push -> cntrl6
- SW5: value SW_Push -> 5x1
- SW6: value SW_Push -> 6x1
- SW7: value SW_Push -> 7x1
- SW8: value SW_Push -> 1x2
- SW9: value SW_Push -> 2x2
- U1: value brain -> brain - teensy 4.0
- U2: value CD74HC4067M -> digital mux - 74hc4067m
- U3: value CD74HC4067M -> analog mux - 74hc4067m
- moved SW36 96.5 mm to (94.0, 118.4), turned to 180 degrees
- moved D36 96.5 mm to (94.0, 126.0)
- moved SW30 83.1 mm to (107.2, 103.3), turned to 180 degrees
- moved D30 83.1 mm to (107.2, 110.9)
- moved D7 81.5 mm to (173.5, 50.8)
- moved SW7 81.5 mm to (173.5, 43.2), turned to 180 degrees
- moved R4 77.9 mm to (91.4, 35.6)
- moved SW29 77.2 mm to (94.0, 103.3), turned to 180 degrees
- moved D29 77.2 mm to (94.0, 110.9)
- moved D24 69.7 mm to (120.5, 95.9)
- moved SW24 69.7 mm to (120.5, 88.3), turned to 180 degrees
- moved SW13 69.2 mm to (160.2, 58.2), turned to 180 degrees
- moved D13 69.2 mm to (160.2, 65.8)
- moved R1 64.5 mm to (82.2, 43.2)
- moved D23 63.7 mm to (107.2, 95.9)
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Connections:
- R1 pad 1: Ctrl1 -> MIDI_IN
- R1 pad 2: 3VDC -> 5VDC
- R2 pad 1: Ctrl2 -> GND
- R2 pad 2: 3VDC -> Net-(R2-Pad2)
- R3 pad 1: Ctrl3 -> Net-(D43-Pad1)
- R3 pad 2: 3VDC -> Net-(J2-Pad4)
- R4 pad 1: Ctrl4 -> 5VDC
- R4 pad 2: 3VDC -> Net-(J3-Pad5)
- SW1 pad 2: 3VDC -> col1
- SW10 pad 2: 3VDC -> col2
- SW11 pad 2: 3VDC -> col2
- SW12 pad 2: 3VDC -> col2
- SW13 pad 2: 3VDC -> col2
- SW14 pad 2: 3VDC -> col2
- SW15 pad 2: 3VDC -> col3
- SW16 pad 2: 3VDC -> col3
- SW17 pad 2: 3VDC -> col3
- SW18 pad 2: 3VDC -> col3
- SW19 pad 2: 3VDC -> col3
- SW2 pad 2: 3VDC -> col1
- SW20 pad 2: 3VDC -> col3
- SW21 pad 2: 3VDC -> col3
- SW22 pad 2: 3VDC -> col4
- SW23 pad 2: 3VDC -> col4
- SW24 pad 2: 3VDC -> col4
- SW25 pad 2: 3VDC -> col4
- SW26 pad 2: 3VDC -> col4
- SW27 pad 2: 3VDC -> col4
- SW28 pad 2: 3VDC -> col4
- SW29 pad 2: 3VDC -> col5
- SW3 pad 2: 3VDC -> col1
- SW30 pad 2: 3VDC -> col5
- SW31 pad 2: 3VDC -> col5
- SW32 pad 2: 3VDC -> col5
- SW33 pad 2: 3VDC -> col5
- SW34 pad 2: 3VDC -> col5
- SW35 pad 2: 3VDC -> col5
- SW36 pad 2: 3VDC -> col6
- SW37 pad 2: 3VDC -> col6
- SW38 pad 2: 3VDC -> col6
- SW39 pad 2: 3VDC -> col6
- SW4 pad 2: 3VDC -> col1
- SW40 pad 2: 3VDC -> col6
- SW41 pad 2: 3VDC -> col6
- SW42 pad 2: 3VDC -> col6
- SW5 pad 2: 3VDC -> col1
- SW6 pad 2: 3VDC -> col1
- SW7 pad 2: 3VDC -> col1
- SW8 pad 2: 3VDC -> col2
- SW9 pad 2: 3VDC -> col2
- U1 pad 10: MuxC1 -> MuxC3
- U1 pad 11: MuxC2 -> MuxC4
- U1 pad 12: MuxC3 -> unconnected-(U1-Pad12)
- U1 pad 2: unconnected-(U1-Pad2) -> MuxR1
- U1 pad 3: unconnected-(U1-Pad3) -> MuxR2
- U1 pad 4: unconnected-(U1-Pad4) -> MuxR3
- U1 pad 5: unconnected-(U1-Pad5) -> MuxR4
- U1 pad 7: MuxR1 -> unconnected-(U1-Pad7)
- U1 pad 8: MuxR2 -> MuxC1
- U1 pad 9: MuxR3 -> MuxC2
- U2 pad 1: GND -> MRR
- U2 pad 10: MRR -> MuxR1
- U2 pad 11: MuxR1 -> MuxR2
- U2 pad 13: MuxR3 -> MuxR4
- U2 pad 14: MuxR2 -> MuxR3
- U2 pad 19: unconnected-(U2-Pad19) -> col6
- U2 pad 2: Ctrl3 -> col1
- U2 pad 20: unconnected-(U2-Pad20) -> col5
- U2 pad 21: unconnected-(U2-Pad21) -> col4
- U2 pad 22: Ctrl1 -> col3
- U2 pad 23: Ctrl2 -> col2
- U3 pad 1: GND -> MRC
- U3 pad 10: MRC -> MuxC1
- U3 pad 11: MuxC1 -> MuxC2
- U3 pad 13: MuxC3 -> MuxC4
- U3 pad 14: MuxC2 -> MuxC3
- U3 pad 2: Ctrl5 -> fp2
- U3 pad 23: Ctrl4 -> main
- U3 pad 4: col6 -> Ctrl5
- U3 pad 5: col5 -> Ctrl4
- U3 pad 6: col4 -> Ctrl3
- U3 pad 7: col3 -> Ctrl2
- U3 pad 8: col2 -> Ctrl1
- U3 pad 9: col1 -> fp1
- U4 pad 6: unconnected-(U4-Pad6) -> GND
Routing:
- net 3VDC: track 0.00 -> 241.5 mm
- net GND: track 104.2 -> 315.2 mm
- net 5VDC: track 28.5 -> 137.6 mm
- net col2: track 0.00 -> 95.4 mm
- net col6: track 0.00 -> 87.5 mm
- net col5: track 0.00 -> 87.5 mm
- net col4: track 0.00 -> 87.5 mm
- net col3: track 0.00 -> 87.5 mm
- net col1: track 0.00 -> 87.0 mm
- net row2: track 0.00 -> 48.5 mm
- net row7: track 0.00 -> 47.8 mm
- net row6: track 0.00 -> 47.8 mm
- net row5: track 0.00 -> 47.8 mm
- net row4: track 0.00 -> 47.8 mm
- net row3: track 0.00 -> 47.8 mm
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Other:
- board outline added: 165.1 x 134.6 mm
- board text added: "MOAR k NOBS - 42"

Commit message: moar brd
Parts:
- added C2: 470uF, Capacitor_THT:C_Disc_D3.4mm_W2.1mm_P2.50mm, F.Cu at (48.3, 109.2)
- J1: footprint Button_Switch_Keyboard:SW_Cherry_MX_2.00u_PCB -> Connector_BarrelJack:BarrelJack_GCT_DCJ200-10-A_Horizontal
- moved J1 11.7 mm to (35.6, 31.8), turned to 180 degrees
- moved J4 2.54 mm to (106.7, 22.9)
- moved J5 2.54 mm to (119.3, 22.9)
- moved J6 2.54 mm to (132.0, 22.9)
- moved J7 2.54 mm to (144.7, 22.9)
- moved J8 2.54 mm to (157.4, 22.9)
- moved J9 2.54 mm to (170.1, 22.9)
Connections:
- D1 pad 1: Net-(D1-Pad1) -> 5VDC
- D10 pad 1: Net-(D10-Pad1) -> Net-(D9-Pad3)
- D11 pad 1: Net-(D11-Pad1) -> Net-(D10-Pad3)
- D12 pad 1: Net-(D12-Pad1) -> Net-(D11-Pad3)
- D12 pad 3: Net-(D1-Pad1) -> Net-(D13-Pad1)
- D13 pad 3: Net-(D12-Pad1) -> Net-(D14-Pad1)
- D14 pad 1: Net-(D11-Pad3) -> Net-(D14-Pad1)
- D15 pad 1: Net-(D15-Pad1) -> Net-(D14-Pad3)
- D15 pad 3: Net-(D10-Pad1) -> Net-(D15-Pad3)
- D16 pad 1: Net-(D16-Pad1) -> Net-(D15-Pad3)
- D17 pad 1: Net-(D17-Pad1) -> Net-(D16-Pad3)
- D17 pad 3: Net-(D17-Pad3) -> Net-(D18-Pad1)
- D2 pad 3: Net-(D11-Pad1) -> Net-(D2-Pad3)
- D20 pad 1: Net-(D20-Pad1) -> Net-(D19-Pad3)
- D20 pad 3: Net-(D17-Pad1) -> Net-(D21-Pad1)
- D21 pad 1: Net-(D16-Pad3) -> Net-(D21-Pad1)
- D21 pad 3: Net-(D21-Pad3) -> Net-(D22-Pad1)
- D22 pad 3: Net-(D15-Pad1) -> Net-(D23-Pad1)
- D23 pad 1: Net-(D14-Pad3) -> Net-(D23-Pad1)
- D23 pad 3: Net-(D23-Pad3) -> Net-(D24-Pad1)
- D24 pad 3: Net-(D13-Pad1) -> Net-(D24-Pad3)
- D25 pad 1: Net-(D25-Pad1) -> Net-(D24-Pad3)
- D25 pad 3: Net-(D24-Pad1) -> Net-(D26-Pad1)
- D26 pad 1: Net-(D23-Pad3) -> Net-(D26-Pad1)
- D27 pad 1: Net-(D27-Pad1) -> Net-(D26-Pad3)
- D27 pad 3: Net-(D22-Pad1) -> Net-(D28-Pad1)
- D28 pad 1: Net-(D21-Pad3) -> Net-(D28-Pad1)
- D29 pad 1: Net-(D29-Pad1) -> Net-(D28-Pad3)
- D29 pad 3: Net-(D20-Pad1) -> Net-(D30-Pad1)
- D3 pad 1: Net-(D10-Pad3) -> Net-(D2-Pad3)
- D30 pad 1: Net-(D19-Pad3) -> Net-(D30-Pad1)
- D32 pad 1: Net-(D32-Pad1) -> Net-(D31-Pad3)
- D32 pad 3: Net-(D29-Pad1) -> Net-(D33-Pad1)
- D33 pad 1: Net-(D28-Pad3) -> Net-(D33-Pad1)
- D33 pad 3: Net-(D33-Pad3) -> Net-(D34-Pad1)
- D34 pad 3: Net-(D27-Pad1) -> Net-(D35-Pad1)
- D35 pad 1: Net-(D26-Pad3) -> Net-(D35-Pad1)
- D36 pad 1: Net-(D36-Pad1) -> Net-(D35-Pad3)
- D36 pad 3: Net-(D25-Pad1) -> Net-(D36-Pad3)
- D37 pad 1: 5VDC -> Net-(D36-Pad3)
- D37 pad 3: Net-(D36-Pad1) -> Net-(D38-Pad1)
- D38 pad 1: Net-(D35-Pad3) -> Net-(D38-Pad1)
- D39 pad 3: Net-(D34-Pad1) -> Net-(D40-Pad1)
- D40 pad 1: Net-(D33-Pad3) -> Net-(D40-Pad1)
- D41 pad 3: Net-(D32-Pad1) -> Net-(D42-Pad1)
- D42 pad 1: Net-(D31-Pad3) -> Net-(D42-Pad1)
- D5 pad 1: Net-(D5-Pad1) -> Net-(D4-Pad3)
- D7 pad 3: Net-(D18-Pad1) -> Net-(D7-Pad3)
- D8 pad 1: Net-(D17-Pad3) -> Net-(D7-Pad3)
- D8 pad 3: Net-(D5-Pad1) -> Net-(D8-Pad3)
- D9 pad 1: Net-(D4-Pad3) -> Net-(D8-Pad3)
- D9 pad 3: Net-(D16-Pad1) -> Net-(D9-Pad3)
Routing:
- net GND: track 315.2 -> 533.8 mm, vias 0 -> 4
- net row7: track 47.8 -> 249.6 mm, vias 0 -> 2
- net E6: track 0.00 -> 198.7 mm
- net E5: track 0.00 -> 178.1 mm
- net E4: track 0.00 -> 155.8 mm
- net row1: track 47.8 -> 190.6 mm, vias 0 -> 8
- net E3: track 0.00 -> 135.7 mm
- net row3: track 47.8 -> 178.0 mm, vias 0 -> 9
- net row6: track 47.8 -> 171.1 mm, vias 0 -> 2
- net row5: track 47.8 -> 162.0 mm, vias 0 -> 3
- net E2: track 0.00 -> 109.1 mm
- net Net-(D28-Pad3): track 0.00 -> 99.3 mm, vias 0 -> 2
- net Net-(D22-Pad1): track 0.00 -> 97.2 mm, vias 0 -> 2
- net Net-(D14-Pad2): track 0.00 -> 96.4 mm, vias 0 -> 2
- net Net-(D14-Pad3): track 0.00 -> 95.8 mm, vias 0 -> 2
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Other:
- board text added: "MOARkNOBS-42"
- board text added: "v2"

Commit message: brd v2
second test
Routing:
- net row4: track 53.9 -> 221.9 mm, vias 1 -> 14
- net row5: track 162.0 -> 255.7 mm, vias 3 -> 13
- net col4: track 87.5 -> 180.2 mm, vias 0 -> 2
- net col6: track 87.5 -> 170.7 mm, vias 0 -> 5
- net col3: track 87.5 -> 168.7 mm, vias 0 -> 6
- net row2: track 122.8 -> 201.9 mm, vias 4 -> 12
- net MuxC4: track 0.00 -> 77.3 mm, vias 0 -> 3
- net row6: track 171.1 -> 246.4 mm, vias 2 -> 10
- net MuxC3: track 0.00 -> 67.4 mm, vias 0 -> 3
- net MuxC1: track 0.00 -> 62.2 mm, vias 0 -> 3
- net MuxC2: track 0.00 -> 60.6 mm, vias 0 -> 3
- net col5: track 87.5 -> 141.1 mm, vias 0 -> 6
- net MIDI_OUT: track 0.00 -> 39.0 mm, vias 0 -> 2
- net row3: track 178.0 -> 215.6 mm, vias 9 -> 13
- net Net-(D18-Pad2): track 0.00 -> 28.0 mm, vias 0 -> 2
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
Commit message: resistors for pull up
Parts:
- added R10: 10k, Resistor_THT:R_Axial_DIN0204_L3.6mm_D1.6mm_P2.54mm_Vertical, B.Cu at (61.0, 66.0)
- added R11: 10k, Resistor_THT:R_Axial_DIN0204_L3.6mm_D1.6mm_P2.54mm_Vertical, F.Cu at (28.4, 109.2)
- added R12: 10k, Resistor_THT:R_Axial_DIN0204_L3.6mm_D1.6mm_P2.54mm_Vertical, F.Cu at (17.3, 106.1)
- added R13: 10k, Resistor_THT:R_Axial_DIN0204_L3.6mm_D1.6mm_P2.54mm_Vertical, F.Cu at (34.0, 99.8)
- added R14: 10k, Resistor_THT:R_Axial_DIN0204_L3.6mm_D1.6mm_P2.54mm_Vertical, F.Cu at (17.3, 99.8)
- added R15: 10k, Resistor_THT:R_Axial_DIN0204_L3.6mm_D1.6mm_P2.54mm_Vertical, F.Cu at (17.3, 102.9)
- added R16: 10k, Resistor_THT:R_Axial_DIN0204_L3.6mm_D1.6mm_P2.54mm_Vertical, F.Cu at (28.4, 102.9)
- added R17: 10k, Resistor_THT:R_Axial_DIN0204_L3.6mm_D1.6mm_P2.54mm_Vertical, F.Cu at (28.4, 106.1)
- added R18: 10k, Resistor_THT:R_Axial_DIN0204_L3.6mm_D1.6mm_P2.54mm_Vertical, F.Cu at (22.9, 106.1)
- added R5: 10k, Resistor_THT:R_Axial_DIN0204_L3.6mm_D1.6mm_P2.54mm_Vertical, F.Cu at (48.3, 73.7)
- added R6: 10k, Resistor_THT:R_Axial_DIN0204_L3.6mm_D1.6mm_P2.54mm_Vertical, F.Cu at (22.9, 91.4)
- added R6: 10k, Resistor_THT:R_Axial_DIN0204_L3.6mm_D1.6mm_P2.54mm_Vertical, B.Cu at (60.9, 63.5)
- added R7: 10k, Resistor_THT:R_Axial_DIN0204_L3.6mm_D1.6mm_P2.54mm_Vertical, F.Cu at (63.5, 73.7)
- added R8: 10k, Resistor_THT:R_Axial_DIN0204_L3.6mm_D1.6mm_P2.54mm_Vertical, F.Cu at (47.5, 62.0)
- added R9: 10k, Resistor_THT:R_Axial_DIN0204_L3.6mm_D1.6mm_P2.54mm_Vertical, F.Cu at (20.3, 86.4)
Routing:
- net 3VDC: track 290.5 -> 391.9 mm, vias 4 -> 8
- net MuxC3: track 67.4 -> 0.00 mm, vias 3 -> 0
- net Net-(D17-Pad2): track 20.1 -> 48.1 mm, vias 0 -> 2
- net Net-(D18-Pad2): track 28.0 -> 0.00 mm, vias 2 -> 0
- net row4: track 221.9 -> 246.3 mm, vias 14 -> 15
- net LED: track 22.9 -> 0.00 mm
- net 5VDC: track 176.8 -> 199.7 mm
- net Net-(D24-Pad2): track 20.2 -> 42.6 mm
- net Net-(D23-Pad2): track 22.4 -> 0.00 mm
- net Net-(D33-Pad2): track 20.9 -> 41.1 mm
- net Net-(D34-Pad2): track 20.2 -> 0.00 mm
- net Net-(D11-Pad2): track 20.2 -> 0.00 mm
- net Net-(D10-Pad2): track 20.2 -> 40.4 mm
- net Net-(D36-Pad2): track 20.7 -> 40.4 mm
- net Net-(D37-Pad2): track 19.6 -> 0.00 mm
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Other:
- board text added: "1x1"
- board text added: "7x6"
- board text added: "EF1"
- board text added: "EF2"
- board text added: "EF3"
- board text added: "EF4"
- board text added: "EF5"
- board text added: "EF6"
- board text added: "MAIN"
- board text added: "MIDI IN"
- board text added: "MIDI OUT"
- board text added: "PWR"
- board text added: "\ | / CNTRL / | \"
- board text added: "brain"
- board text added: "f1"
- board text added: "f2"

Commit message: reorg
Parts:
- removed the C2 at (83.8, 38.1)
- removed the C2 at (48.3, 109.2)
- removed the R6 at (22.9, 91.4)
- removed the R6 at (60.9, 63.5)
- added C2: 470uF, Capacitor_THT:C_Disc_D3.4mm_W2.1mm_P2.50mm, F.Cu at (73.7, 134.6)
- added R6: 10k, Resistor_THT:R_Axial_DIN0204_L3.6mm_D1.6mm_P2.54mm_Vertical, F.Cu at (43.8, 85.9)
- R10: moved to F.Cu
- moved C3 61.5 mm to (17.5, 109.2)
- moved U2 43.3 mm to (27.9, 91.4)
- moved R12 40.5 mm to (50.8, 83.4)
- moved U3 40.2 mm to (27.9, 109.2)
- moved R15 35.6 mm to (50.8, 91.0)
- moved R14 35.4 mm to (50.8, 88.5)
- moved R10 34.6 mm to (43.8, 96.1)
- moved J10 31.9 mm to (63.5, 72.3)
- moved C4 31.3 mm to (17.4, 83.9)
- moved R8 29.2 mm to (43.8, 91.0), turned to 0 degrees
- moved R18 28.9 mm to (50.8, 98.6)
- moved R1 26.9 mm to (55.9, 48.7)
- moved R7 24.7 mm to (43.8, 88.5), turned to 0 degrees
- moved R9 24.5 mm to (43.8, 93.5)
- moved R17 24.5 mm to (50.8, 96.1)
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Routing:
- net 3VDC: track 391.9 -> 238.6 mm, vias 8 -> 3
- net 5VDC: track 199.7 -> 100.9 mm, vias 1 -> 0
- net GND: track 544.1 -> 480.2 mm, vias 6 -> 4
- net row5: track 272.5 -> 215.2 mm, vias 13 -> 11
- net Ctrl3: track 91.1 -> 35.1 mm, vias 2 -> 1
- net SCL: track 61.6 -> 6.30 mm
- net Ctrl2: track 67.3 -> 13.4 mm, vias 4 -> 1
- net LEDcntrl: track 56.9 -> 5.04 mm, vias 2 -> 1
- net Ctrl5: track 64.6 -> 16.0 mm, vias 4 -> 1
- net row2: track 201.9 -> 153.9 mm
- net Ctrl6: track 66.1 -> 18.5 mm, vias 7 -> 3
- net row4: track 246.3 -> 202.7 mm, vias 15 -> 12
- net Net-(D24-Pad2): track 42.6 -> 0.00 mm
- net Net-(D23-Pad2): track 0.00 -> 42.6 mm
- net row7: track 250.0 -> 209.3 mm, vias 2 -> 1
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